File: Electrical/Common/Common.sch (KiCad schematic (older format))
At the start: 62 parts, among them J201 01x02, J202 01x04, J203 01x03, J204 01x04, J205 01x03, J206 USB_OTG, J207 01x04, J208 01x02, J209 01x04, J210 01x02, J211 01x02, J212 4PostTerm, J213 2PostTerm, J214 2PostTerm, J215 JST_3, Q201 FDC6420C, Q202 FDG1024NZ, U201 TPD4S012, U202 ACS712ELCTR-05B-T, U203 ACS712ELCTR-05B-T, U204 24LC256, U205 LM2576HVS-ADJ, U206 LM2576HVS-ADJ

Commit message: Fixed issues with socket strips vs pin headers
Parts:
- J201, J208, J210, J211: footprint Socket_Strips:Socket_Strip_Straight_1x02_Pitch2.54mm -> Pin_Headers:Pin_Header_Straight_1x02_Pitch2.54mm
- J202, J204, J207, J209, JP201: footprint Socket_Strips:Socket_Strip_Straight_1x04_Pitch2.54mm -> Pin_Headers:Pin_Header_Straight_1x04_Pitch2.54mm
- J203, J205: footprint Socket_Strips:Socket_Strip_Straight_1x03_Pitch2.54mm -> Pin_Headers:Pin_Header_Straight_1x03_Pitch2.54mm
- JP208, JP209: footprint Socket_Strips:Socket_Strip_Straight_2x04_Pitch2.54mm -> Pin_Headers:Pin_Header_Straight_1x08_Pitch2.54mm
Changed lines of the file:
@@
 F 0 "J208" H 6200 3350 50  0000 C CNN
 F 1 "01x02" V 6300 3200 50  0000 C CNN
-F 2 "Socket_Strips:Socket_Strip_Straight_1x02_Pitch2.54mm" H 6200 3250 50  0001 C CNN
+F 2 "Pin_Headers:Pin_Header_Straight_1x02_Pitch2.54mm" H 6200 3250 50  0001 C CNN
 F 3 "" H 6200 3250 50  0001 C CNN
 	1    6200 3250
@@
 F 0 "J201" H 3400 1350 50  0000 C CNN
 F 1 "01x02" V 3250 1350 50  0000 C CNN
-F 2 "Socket_Strips:Socket_Strip_Straight_1x02_Pitch2.54mm" H 3150 1400 50  0001 C CNN
+F 2 "Pin_Headers:Pin_Header_Straight_1x02_Pitch2.54mm" H 3150 1400 50  0001 C CNN
 F 3 "" H 3150 1400 50  0001 C CNN
 	1    3150 1400
@@
 F 0 "J204" H 3950 7050 50  0000 C CNN
 F 1 "01x04" V 4050 6800 50  0000 C CNN
-F 2 "Socket_Strips:Socket_Strip_Straight_1x04_Pitch2.54mm" H 3950 6850 50  0001 C CNN
+F 2 "Pin_Headers:Pin_Header_Straight_1x04_Pitch2.54mm" H 3950 6850 50  0001 C CNN
 F 3 "" H 3950 6850 50  0001 C CNN
 	1    3950 6850
@@
 F 0 "J202" H 3200 5250 50  0000 C CNN
 F 1 "01x04" V 3300 5000 50  0000 C CNN
-F 2 "Socket_Strips:Socket_Strip_Straight_1x04_Pitch2.54mm" H 3200 5050 50  0001 C CNN
+F 2 "Pin_Headers:Pin_Header_Straight_1x04_Pitch2.54mm" H 3200 5050 50  0001 C CNN
 F 3 "" H 3200 5050 50  0001 C CNN
 	1    3200 5050
@@
 F 0 "JP201" V 3100 7450 50  0000 L CNN
 F 1 "01x04" V 3200 7250 50  0000 C CNN
-F 2 "Socket_Strips:Socket_Strip_Straight_1x04_Pitch2.54mm" H 3100 7300 50  0001 C CNN
+F 2 "Pin_Headers:Pin_Header_Straight_1x04_Pitch2.54mm" H 3100 7300 50  0001 C CNN
 F 3 "" H 3100 7300 50  0001 C CNN
 	1    3100 7300
@@
 F 0 "J207" H 4900 7000 50  0000 C CNN
 F 1 "01x04" V 5000 6750 50  0000 C CNN
-F 2 "Socket_Strips:Socket_Strip_Straight_1x04_Pitch2.54mm" H 4900 6800 50  0001 C CNN
+F 2 "Pin_Headers:Pin_Header_Straight_1x04_Pitch2.54mm" H 4900 6800 50  0001 C CNN
 F 3 "" H 4900 6800 50  0001 C CNN
 	1    4900 6800
@@
 F 0 "J209" H 6600 7600 50  0000 C CNN
 F 1 "01x04" V 6700 7350 50  0000 C CNN
-F 2 "Socket_Strips:Socket_Strip_Straight_1x04_Pitch2.54mm" H 6600 7400 50  0001 C CNN
+F 2 "Pin_Headers:Pin_Header_Straight_1x04_Pitch2.54mm" H 6600 7400 50  0001 C CNN
 F 3 "" H 6600 7400 50  0001 C CNN
 	1    6600 7400
@@
 F 0 "J210" H 6950 1050 50  0000 C CNN
 F 1 "01x02" V 7050 900 50  0000 C CNN
-F 2 "Socket_Strips:Socket_Strip_Straight_1x02_Pitch2.54mm" H 6950 950 50  0001 C CNN
+F 2 "Pin_Headers:Pin_Header_Straight_1x02_Pitch2.54mm" H 6950 950 50  0001 C CNN
 F 3 "" H 6950 950 50  0001 C CNN
 	1    6950 950
@@
 F 0 "J211" H 7250 3350 50  0000 C CNN
 F 1 "01x02" V 7350 3200 50  0000 C CNN
-F 2 "Socket_Strips:Socket_Strip_Straight_1x02_Pitch2.54mm" H 7250 3250 50  0001 C CNN
+F 2 "Pin_Headers:Pin_Header_Straight_1x02_Pitch2.54mm" H 7250 3250 50  0001 C CNN
 F 3 "" H 7250 3250 50  0001 C CNN
 	1    7250 3250
@@
 F 0 "J205" H 4000 6350 50  0000 C CNN
 F 1 "01x03" V 4100 6150 50  0000 C CNN
-F 2 "Socket_Strips:Socket_Strip_Straight_1x03_Pitch2.54mm" H 4000 6150 50  0001 C CNN
+F 2 "Pin_Headers:Pin_Header_Straight_1x03_Pitch2.54mm" H 4000 6150 50  0001 C CNN
 F 3 "" H 4000 6150 50  0001 C CNN
 	1    4000 6150
@@
 F 0 "J203" H 3500 4500 50  0000 C CNN
 F 1 "01x03" V 3600 4300 50  0000 C CNN
-F 2 "Socket_Strips:Socket_Strip_Straight_1x03_Pitch2.54mm" H 3500 4300 50  0001 C CNN
+F 2 "Pin_Headers:Pin_Header_Straight_1x03_Pitch2.54mm" H 3500 4300 50  0001 C CNN
 F 3 "" H 3500 4300 50  0001 C CNN
 	1    3500 4300
@@
 F 0 "JP209" H 6350 6400 50  0000 C CNN
 F 1 "02x04" H 6350 5900 50  0000 C CNN
-F 2 "Socket_Strips:Socket_Strip_Straight_2x04_Pitch2.54mm" H 6300 6200 50  0001 C CNN
+F 2 "Pin_Headers:Pin_Header_Straight_1x08_Pitch2.54mm" H 6300 6200 50  0001 C CNN
 F 3 "" H 6300 6200 50  0001 C CNN
 	1    6300 6200
@@
 F 0 "JP208" H 6250 5300 50  0000 C CNN
 F 1 "02x04" H 6250 4800 50  0000 C CNN
-F 2 "Socket_Strips:Socket_Strip_Straight_2x04_Pitch2.54mm" H 6200 5100 50  0001 C CNN
+F 2 "Pin_Headers:Pin_Header_Straight_1x08_Pitch2.54mm" H 6200 5100 50  0001 C CNN
 F 3 "" H 6200 5100 50  0001 C CNN
 	1    6200 5100

Commit message: Working on layout and routing.
Parts:
- removed C206: 100uF, Capacitors_SMD:CP_Elec_8x10, symbol CP1
- added J216, J217: 2PostTerm, footprints:TerminalBlock_Custom_1x02.54mm, symbol Screw_Terminal_01x02
- added MK201, MK202, MK203, MK204: Mounting_Hole_PAD, Mounting_Holes:MountingHole_3.2mm_M3_ISO14580_Pad, symbol Mounting_Hole_PAD
- added RN207: 1K2, footprints:R_Array_1206x04, symbol R_Pack04
- C207: value 100uF -> 1000uF
- J202, J204: footprint Pin_Headers:Pin_Header_Straight_1x04_Pitch2.54mm -> footprints:Molex-SL-4POS
- J203, J205: footprint Pin_Headers:Pin_Header_Straight_1x03_Pitch2.54mm -> Connectors_JST:JST_XH_B03B-XH-A_03x2.50mm_Straight
- JP208, JP209: footprint Pin_Headers:Pin_Header_Straight_1x08_Pitch2.54mm -> footprints:Pin_Header_Straight_2x04_Pitch2.54mm_AB
- U205, U206: footprint TO_SOT_Packages_SMD:TO-263-5Lead -> TO_SOT_Packages_SMD:TO-263-5_TabPin3
Connections:
- net labels added: usb1_d+, usb1_d-
- net labels removed: usb1_dn, usb1_dp
- wire segments 240 -> 263
Other:
- moved on the sheet: J210, J213, J214, J215, JP202, JP203, JP204, JP205, JP206, JP207, JP210, JP211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
