File: Electrical/Common/Common.sch (KiCad schematic (older format))
At the start: 76 parts, among them J201 01x03, J202 01x04, J203 01x03, J204 01x04, J205 01x03, J206 USB_OTG, J207 01x04, J208 01x02, J209 01x04, J210 01x02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

Commit message: Rearranged the power outputs to support TE Connectivity AMP connectors.
Connections:
- wire segments 289 -> 290
Changed lines of the file:
@@
 LIBS:allegro
 LIBS:mechanical
-LIBS:Quad-cache
+LIBS:Dual-cache
 EELAYER 25 0
 EELAYER END
 $Descr A4 11693 8268
 encoding utf-8
-Sheet 2 6
+Sheet 2 4
 Title ""
 Date ""
@@
 Text Label 4500 2650 1    60   ~ 0
 usb1_5V
-Text Label 5300 2650 1    60   ~ 0
+Text Label 5450 2250 1    60   ~ 0
 usb1_vbus
 $Comp
@@
 	3950 3250 3950 3450
 Wire Wire Line
-	4800 2650 5300 2650
-Wire Wire Line
-	4350 2650 4600 2650
+	4350 2650 5300 2650
 Wire Wire Line
 	2800 2150 2800 2250
@@
 Wire Wire Line
 	4900 2450 4900 2400
-Wire Wire Line
-	5200 2200 5200 2650
 Wire Wire Line
 	2800 2600 3050 2600
@@
 L Ferrite_Bead_Small FB202
 U 1 1 5A7E3264
-P 4700 2650
-F 0 "FB202" H 4775 2700 50  0000 L CNN
-F 1 "120" H 4775 2600 50  0000 L CNN
-F 2 "SMD_Packages:SMD-1206_Pol" V 4630 2650 50  0001 C CNN
-F 3 "" H 4700 2650 50  0001 C CNN
-	1    4700 2650
-	0    -1   -1   0
+P 5200 2450
+F 0 "FB202" H 5275 2500 50  0000 L CNN
+F 1 "120" H 5275 2400 50  0000 L CNN
+F 2 "SMD_Packages:SMD-1206_Pol" V 5130 2450 50  0001 C CNN
+F 3 "" H 5200 2450 50  0001 C CNN
+	1    5200 2450
+	1    0    0    -1
 $EndComp
 $Comp
@@
 F 3 "" H 4050 3450 50  0001 C CNN
 	1    4050 3450
-	0    -1   -1   0
-$EndComp
+	0    1    -1   0
+$EndComp
+Wire Wire Line
+	5450 2250 5200 2250
+Connection ~ 5200 2250
+Wire Wire Line
+	5200 2650 5200 2550
+Wire Wire Line
+	5200 2200 5200 2350
 $EndSCHEMATC
