File: Electrical/Common/Stepper.sch (KiCad schematic (older format))
At the start: 12 parts, among them Q201 FDC6420C

Commit message: Completed components common to both quad and dual steppers (with the exception of power breakouts)
Changed lines of the file:
@@
 LIBS:dc-dc
 LIBS:IC
+LIBS:tpd4s012
 LIBS:Common-cache
 EELAYER 25 0
@@
 AR Path="/5A50EA77/5A50EABF" Ref="A201"  Part="1"
 AR Path="/5A569D3F/5A50EABF" Ref="A301"  Part="1"
-F 0 "A201" H 2650 4200 50  0000 R CNN
+F 0 "A301" H 2650 4200 50  0000 R CNN
 F 1 "Pololu_Breakout_A4988" H 2650 4100 50  0000 R CNN
 F 2 "Modules:Pololu_Breakout-16_15.2x20.3mm" H 3025 2700 50  0001 L CNN
@@
 AR Path="/5A50EA77/5A50EB28" Ref="A202"  Part="1"
 AR Path="/5A569D3F/5A50EB28" Ref="A302"  Part="1"
-F 0 "A202" H 4650 4050 50  0000 R CNN
+F 0 "A302" H 4650 4050 50  0000 R CNN
 F 1 "Pololu_Breakout_DRV8825" H 4650 3950 50  0000 R CNN
 F 2 "Modules:Pololu_Breakout-16_15.2x20.3mm" H 4950 2600 50  0001 L CNN
@@
 AR Path="/5A50EA77/5A50F831" Ref="A203"  Part="1"
 AR Path="/5A569D3F/5A50F831" Ref="A303"  Part="1"
-F 0 "A203" H 6650 4350 50  0000 R CNN
+F 0 "A303" H 6650 4350 50  0000 R CNN
 F 1 "Pololu_Breakout_DRV8834" H 6650 4250 50  0000 R CNN
 F 2 "Modules:Pololu_Breakout-16_15.2x20.3mm" H 6950 2700 50  0001 L CNN
@@
 AR Path="/5A50EA77/5A50F8CE" Ref="A204"  Part="1"
 AR Path="/5A569D3F/5A50F8CE" Ref="A304"  Part="1"
-F 0 "A204" H 8600 4350 50  0000 R CNN
+F 0 "A304" H 8600 4350 50  0000 R CNN
 F 1 "Pololu_Breakout_DRV8880" H 8600 4250 50  0000 R CNN
 F 2 "Modules:Pololu_Breakout-16_15.2x20.3mm" H 8900 2700 50  0001 L CNN
@@
 	1    0    0    -1
 $EndComp
-Text HLabel 3250 3350 2    60   Input ~ 0
+Text HLabel 3250 3350 2    60   Output ~ 0
 A2
-Text HLabel 3250 3450 2    60   Input ~ 0
+Text HLabel 3250 3450 2    60   Output ~ 0
 A1
-Text HLabel 3250 3550 2    60   Input ~ 0
+Text HLabel 3250 3550 2    60   Output ~ 0
 B1
-Text HLabel 3250 3650 2    60   Input ~ 0
+Text HLabel 3250 3650 2    60   Output ~ 0
 B2
-Text HLabel 5150 3400 2    60   Input ~ 0
+Text HLabel 5150 3400 2    60   Output ~ 0
 A2
-Text HLabel 5150 3300 2    60   Input ~ 0
+Text HLabel 5150 3300 2    60   Output ~ 0
 A1
-Text HLabel 5150 3600 2    60   Input ~ 0
+Text HLabel 5150 3600 2    60   Output ~ 0
 B1
-Text HLabel 5150 3700 2    60   Input ~ 0
+Text HLabel 5150 3700 2    60   Output ~ 0
 B2
-Text HLabel 7150 3400 2    60   Input ~ 0
+Text HLabel 7150 3400 2    60   Output ~ 0
 A2
-Text HLabel 7150 3300 2    60   Input ~ 0
+Text HLabel 7150 3300 2    60   Output ~ 0
 A1
-Text HLabel 7150 3600 2    60   Input ~ 0
+Text HLabel 7150 3600 2    60   Output ~ 0
 B1
-Text HLabel 7150 3700 2    60   Input ~ 0
+Text HLabel 7150 3700 2    60   Output ~ 0
 B2
-Text HLabel 9100 3300 2    60   Input ~ 0
+Text HLabel 9100 3300 2    60   Output ~ 0
 A2
-Text HLabel 9100 3400 2    60   Input ~ 0
+Text HLabel 9100 3400 2    60   Output ~ 0
 A1
-Text HLabel 9100 3600 2    60   Input ~ 0
+Text HLabel 9100 3600 2    60   Output ~ 0
 B1
-Text HLabel 9100 3700 2    60   Input ~ 0
+Text HLabel 9100 3700 2    60   Output ~ 0
 B2
 Text HLabel 8300 3200 0    60   Input ~ 0
@@
 AR Path="/5A50EA77/5A50FF78" Ref="#PWR205"  Part="1"
 AR Path="/5A569D3F/5A50FF78" Ref="#PWR305"  Part="1"
-F 0 "#PWR205" H 8800 4100 50  0001 C CNN
+F 0 "#PWR305" H 8800 4100 50  0001 C CNN
 F 1 "GND" H 8800 4200 50  0000 C CNN
 F 2 "" H 8800 4350 50  0001 C CNN
@@
 AR Path="/5A50EA77/5A50FFB9" Ref="#PWR204"  Part="1"
 AR Path="/5A569D3F/5A50FFB9" Ref="#PWR304"  Part="1"
-F 0 "#PWR204" H 6950 4100 50  0001 C CNN
+F 0 "#PWR304" H 6950 4100 50  0001 C CNN
 F 1 "GND" H 6950 4200 50  0000 C CNN
 F 2 "" H 6950 4350 50  0001 C CNN
@@
 AR Path="/5A50EA77/5A50FFD0" Ref="#PWR203"  Part="1"
 AR Path="/5A569D3F/5A50FFD0" Ref="#PWR303"  Part="1"
-F 0 "#PWR203" H 4850 4000 50  0001 C CNN
+F 0 "#PWR303" H 4850 4000 50  0001 C CNN
 F 1 "GND" H 4850 4100 50  0000 C CNN
 F 2 "" H 4850 4250 50  0001 C CNN
@@
 AR Path="/5A50EA77/5A50FFEF" Ref="#PWR201"  Part="1"
 AR Path="/5A569D3F/5A50FFEF" Ref="#PWR301"  Part="1"
-F 0 "#PWR201" H 2950 4050 50  0001 C CNN
+F 0 "#PWR301" H 2950 4050 50  0001 C CNN
 F 1 "GND" H 2950 4150 50  0000 C CNN
 F 2 "" H 2950 4300 50  0001 C CNN
@@
 AR Path="/5A50EA77/5A510065" Ref="JP201"  Part="1"
 AR Path="/5A569D3F/5A510065" Ref="JP301"  Part="1"
-F 0 "JP201" H 1850 1350 50  0000 C CNN
+F 0 "JP301" H 1850 1350 50  0000 C CNN
 F 1 "01x03" H 1850 950 50  0000 C CNN
 F 2 "" H 1850 1150 50  0001 C CNN
@@
 AR Path="/5A50EA77/5A5103B4" Ref="JP203"  Part="1"
 AR Path="/5A569D3F/5A5103B4" Ref="JP303"  Part="1"
-F 0 "JP203" H 9850 1150 50  0000 C CNN
+F 0 "JP303" H 9850 1150 50  0000 C CNN
 F 1 "01x02" H 9850 850 50  0000 C CNN
 F 2 "" H 9850 1050 50  0001 C CNN
@@
 AR Path="/5A50EA77/5A559C1C" Ref="Q201"  Part="2"
 AR Path="/5A569D3F/5A559C1C" Ref="Q301"  Part="2"
-F 0 "Q201" H 4950 6725 50  0000 L CNN
+F 0 "Q301" H 4950 6725 50  0000 L CNN
 F 1 "FDC6420C" H 4950 6650 50  0000 L CNN
 F 2 "TO_SOT_Packages_SMD:SOT-363_SC-70-6" H 4950 6575 50  0001 L CIN
@@
 AR Path="/5A50EA77/5A559D2E" Ref="Q201"  Part="1"
 AR Path="/5A569D3F/5A559D2E" Ref="Q301"  Part="1"
-F 0 "Q201" H 3800 6025 50  0000 L CNN
+F 0 "Q301" H 3800 6025 50  0000 L CNN
 F 1 "FDC6420C" H 3800 5950 50  0000 L CNN
 F 2 "TO_SOT_Packages_SMD:SOT-363_SC-70-6" H 3800 5875 50  0001 L CIN
@@
 AR Path="/5A50EA77/5A559FB3" Ref="R202"  Part="1"
 AR Path="/5A569D3F/5A559FB3" Ref="R302"  Part="1"
-F 0 "R202" V 3880 5550 50  0000 C CNN
+F 0 "R302" V 3880 5550 50  0000 C CNN
 F 1 "12K" V 3800 5550 50  0000 C CNN
 F 2 "" V 3730 5550 50  0001 C CNN
@@
 AR Path="/5A50EA77/5A55A014" Ref="R204"  Part="1"
 AR Path="/5A569D3F/5A55A014" Ref="R304"  Part="1"
-F 0 "R204" V 4630 6850 50  0000 C CNN
+F 0 "R304" V 4630 6850 50  0000 C CNN
 F 1 "12K" V 4550 6850 50  0000 C CNN
 F 2 "" V 4480 6850 50  0001 C CNN
@@
 AR Path="/5A50EA77/5A55A0AD" Ref="R203"  Part="1"
 AR Path="/5A569D3F/5A55A0AD" Ref="R303"  Part="1"
-F 0 "R203" V 3880 6600 50  0000 C CNN
+F 0 "R303" V 3880 6600 50  0000 C CNN
 F 1 "1K2" V 3800 6600 50  0000 C CNN
 F 2 "" V 3730 6600 50  0001 C CNN
@@
 	4550 7000 4850 7000
 Wire Wire Line
-	4550 6600 4550 6700
+	4550 6400 4550 6700
 Wire Wire Line
 	4850 6450 4850 5900
@@
 AR Path="/5A50EA77/5A55A389" Ref="#PWR202"  Part="1"
 AR Path="/5A569D3F/5A55A389" Ref="#PWR302"  Part="1"
-F 0 "#PWR202" H 4750 6750 50  0001 C CNN
+F 0 "#PWR302" H 4750 6750 50  0001 C CNN
 F 1 "GND" H 4750 6850 50  0000 C CNN
 F 2 "" H 4750 7000 50  0001 C CNN
@@
 AR Path="/5A50EA77/5A55A50D" Ref="R201"  Part="1"
 AR Path="/5A569D3F/5A55A50D" Ref="R301"  Part="1"
-F 0 "R201" V 3580 6350 50  0000 C CNN
+F 0 "R301" V 3580 6350 50  0000 C CNN
 F 1 "22" V 3500 6350 50  0000 C CNN
 F 2 "" V 3430 6350 50  0001 C CNN
@@
 AR Path="/5A50EA77/5A55DB5B" Ref="JP202"  Part="1"
 AR Path="/5A569D3F/5A55DB5B" Ref="JP302"  Part="1"
-F 0 "JP202" H 9450 1280 50  0000 C CNN
+F 0 "JP302" H 9450 1280 50  0000 C CNN
 F 1 "Jmp" H 9460 1140 50  0000 C CNN
 F 2 "" H 9450 1200 50  0001 C CNN
@@
 Text Label 8300 2900 2    60   ~ 0
 fault_supply
-Text HLabel 4550 6600 1    60   Input ~ 0
+Text HLabel 4550 6400 1    60   Output ~ 0
 ~FLT
 $EndSCHEMATC

Commit message: Completed Schematic for Dual implementation
Parts:
- removed JP201: 01x03, symbol Conn_01x03
- removed JP203: 01x02, symbol Conn_01x02
- removed Q201: FDC6420C, TO_SOT_Packages_SMD:SOT-363_SC-70-6, symbol FDC6420C
- removed R201: 22, symbol R
- added JP401: 01x03, symbol Conn_01x03
- added JP403: 01x02, symbol Conn_01x02
- added Q401: FDC6420C, TO_SOT_Packages_SMD:SOT-363_SC-70-6, symbol FDC6420C
- added R401: 22, symbol R
- renumbered A201 to A401, A202 to A402, A203 to A403, A204 to A404, JP202 to JP402, R202 to R402, R203 to R403, R204 to R404
Connections:
- net 3V3S: now also JP403.1 (Pin_1), Q401.6 (S)
- net GND: now also Q401.4 (D)
- net SLP: now also JP403.2 (Pin_2)
- net Vadj: now also JP401.3 (Pin_3)
- net Vin: now also JP401.1 (Pin_1)
- net Vmot: now also JP401.2 (Pin_2)
- net fault_supply: now also R401.1
- net ~FLT: now also Q401.3 (G)
- net at R402.2: now also Q401.1 (G), Q401.2 (S)
- new net: Q401.5 (D), R401.2
Changed lines of the file:
@@
 LIBS:valves
 LIBS:modules
+LIBS:IC
+LIBS:dc-dc
 LIBS:allegro
-LIBS:dc-dc
-LIBS:IC
-LIBS:tpd4s012
-LIBS:Common-cache
+LIBS:Dual-cache
 EELAYER 25 0
 EELAYER END
 $Descr A4 11693 8268
 encoding utf-8
-Sheet 2 3
+Sheet 4 4
 Title ""
 Date ""
@@
 $EndDescr
 $Comp
-L Pololu_Breakout_A4988 A201
+L Pololu_Breakout_A4988 A401
 U 1 1 5A50EABF
 P 2750 3450
-AR Path="/5A50EA77/5A50EABF" Ref="A201"  Part="1"
-AR Path="/5A569D3F/5A50EABF" Ref="A301"  Part="1"
-F 0 "A301" H 2650 4200 50  0000 R CNN
+F 0 "A401" H 2650 4200 50  0000 R CNN
 F 1 "Pololu_Breakout_A4988" H 2650 4100 50  0000 R CNN
 F 2 "Modules:Pololu_Breakout-16_15.2x20.3mm" H 3025 2700 50  0001 L CNN
@@
 $EndComp
 $Comp
-L Pololu_Breakout_DRV8825 A202
+L Pololu_Breakout_DRV8825 A402
 U 1 1 5A50EB28
 P 4750 3400
-AR Path="/5A50EA77/5A50EB28" Ref="A202"  Part="1"
-AR Path="/5A569D3F/5A50EB28" Ref="A302"  Part="1"
-F 0 "A302" H 4650 4050 50  0000 R CNN
+F 0 "A402" H 4650 4050 50  0000 R CNN
 F 1 "Pololu_Breakout_DRV8825" H 4650 3950 50  0000 R CNN
 F 2 "Modules:Pololu_Breakout-16_15.2x20.3mm" H 4950 2600 50  0001 L CNN
@@
 $EndComp
 $Comp
-L Pololu_Breakout_DRV8834 A203
+L Pololu_Breakout_DRV8834 A403
 U 1 1 5A50F831
 P 6750 3500
-AR Path="/5A50EA77/5A50F831" Ref="A203"  Part="1"
-AR Path="/5A569D3F/5A50F831" Ref="A303"  Part="1"
-F 0 "A303" H 6650 4350 50  0000 R CNN
+F 0 "A403" H 6650 4350 50  0000 R CNN
 F 1 "Pololu_Breakout_DRV8834" H 6650 4250 50  0000 R CNN
 F 2 "Modules:Pololu_Breakout-16_15.2x20.3mm" H 6950 2700 50  0001 L CNN
@@
 $EndComp
 $Comp
-L Pololu_Breakout_DRV8880 A204
+L Pololu_Breakout_DRV8880 A404
 U 1 1 5A50F8CE
 P 8700 3500
-AR Path="/5A50EA77/5A50F8CE" Ref="A204"  Part="1"
-AR Path="/5A569D3F/5A50F8CE" Ref="A304"  Part="1"
-F 0 "A304" H 8600 4350 50  0000 R CNN
+F 0 "A404" H 8600 4350 50  0000 R CNN
 F 1 "Pololu_Breakout_DRV8880" H 8600 4250 50  0000 R CNN
 F 2 "Modules:Pololu_Breakout-16_15.2x20.3mm" H 8900 2700 50  0001 L CNN
@@
 DIR
 $Comp
-L GND #PWR205
+L GND #PWR405
 U 1 1 5A50FF78
 P 8800 4350
-AR Path="/5A50EA77/5A50FF78" Ref="#PWR205"  Part="1"
-AR Path="/5A569D3F/5A50FF78" Ref="#PWR305"  Part="1"
-F 0 "#PWR305" H 8800 4100 50  0001 C CNN
+F 0 "#PWR405" H 8800 4100 50  0001 C CNN
 F 1 "GND" H 8800 4200 50  0000 C CNN
 F 2 "" H 8800 4350 50  0001 C CNN
@@
 	8800 4300 8700 4300
 $Comp
-L GND #PWR204
+L GND #PWR404
 U 1 1 5A50FFB9
 P 6950 4350
-AR Path="/5A50EA77/5A50FFB9" Ref="#PWR204"  Part="1"
-AR Path="/5A569D3F/5A50FFB9" Ref="#PWR304"  Part="1"
-F 0 "#PWR304" H 6950 4100 50  0001 C CNN
+F 0 "#PWR404" H 6950 4100 50  0001 C CNN
 F 1 "GND" H 6950 4200 50  0000 C CNN
 F 2 "" H 6950 4350 50  0001 C CNN
@@
 $EndComp
 $Comp
-L GND #PWR203
+L GND #PWR403
 U 1 1 5A50FFD0
 P 4850 4250
-AR Path="/5A50EA77/5A50FFD0" Ref="#PWR203"  Part="1"
-AR Path="/5A569D3F/5A50FFD0" Ref="#PWR303"  Part="1"
-F 0 "#PWR303" H 4850 4000 50  0001 C CNN
+F 0 "#PWR403" H 4850 4000 50  0001 C CNN
 F 1 "GND" H 4850 4100 50  0000 C CNN
 F 2 "" H 4850 4250 50  0001 C CNN
@@
 $EndComp
 $Comp
-L GND #PWR201
-U 1 1 5A50FFEF
+L GND #PWR401
+U 1 1 5A57FC8B
 P 2950 4300
-AR Path="/5A50EA77/5A50FFEF" Ref="#PWR201"  Part="1"
-AR Path="/5A569D3F/5A50FFEF" Ref="#PWR301"  Part="1"
-F 0 "#PWR301" H 2950 4050 50  0001 C CNN
+F 0 "#PWR401" H 2950 4050 50  0001 C CNN
 F 1 "GND" H 2950 4150 50  0000 C CNN
 F 2 "" H 2950 4300 50  0001 C CNN
@@
 Vadj
 $Comp
-L Conn_01x03 JP201
-U 1 1 5A510065
+L Conn_01x03 JP401
+U 1 1 5A57FC8C
 P 1850 1150
-AR Path="/5A50EA77/5A510065" Ref="JP201"  Part="1"
-AR Path="/5A569D3F/5A510065" Ref="JP301"  Part="1"
-F 0 "JP301" H 1850 1350 50  0000 C CNN
+F 0 "JP401" H 1850 1350 50  0000 C CNN
 F 1 "01x03" H 1850 950 50  0000 C CNN
 F 2 "" H 1850 1150 50  0001 C CNN
@@
 Cfg2
 $Comp
-L Conn_01x02 JP203
-U 1 1 5A5103B4
+L Conn_01x02 JP403
+U 1 1 5A57FC8D
 P 9850 1050
-AR Path="/5A50EA77/5A5103B4" Ref="JP203"  Part="1"
-AR Path="/5A569D3F/5A5103B4" Ref="JP303"  Part="1"
-F 0 "JP303" H 9850 1150 50  0000 C CNN
+F 0 "JP403" H 9850 1150 50  0000 C CNN
 F 1 "01x02" H 9850 850 50  0000 C CNN
 F 2 "" H 9850 1050 50  0001 C CNN
@@
 SLP
 $Comp
-L FDC6420C Q201
-U 2 1 5A559C1C
+L FDC6420C Q401
+U 2 1 5A57FC8E
 P 4750 6650
-AR Path="/5A50EA77/5A559C1C" Ref="Q201"  Part="2"
-AR Path="/5A569D3F/5A559C1C" Ref="Q301"  Part="2"
-F 0 "Q301" H 4950 6725 50  0000 L CNN
+F 0 "Q401" H 4950 6725 50  0000 L CNN
 F 1 "FDC6420C" H 4950 6650 50  0000 L CNN
 F 2 "TO_SOT_Packages_SMD:SOT-363_SC-70-6" H 4950 6575 50  0001 L CIN
@@
 $EndComp
 $Comp
-L FDC6420C Q201
-U 1 1 5A559D2E
+L FDC6420C Q401
+U 1 1 5A57FC8F
 P 3600 5950
-AR Path="/5A50EA77/5A559D2E" Ref="Q201"  Part="1"
-AR Path="/5A569D3F/5A559D2E" Ref="Q301"  Part="1"
-F 0 "Q301" H 3800 6025 50  0000 L CNN
+F 0 "Q401" H 3800 6025 50  0000 L CNN
 F 1 "FDC6420C" H 3800 5950 50  0000 L CNN
 F 2 "TO_SOT_Packages_SMD:SOT-363_SC-70-6" H 3800 5875 50  0001 L CIN
@@
 $EndComp
 $Comp
-L R R202
+L R R402
 U 1 1 5A559FB3
 P 3800 5550
-AR Path="/5A50EA77/5A559FB3" Ref="R202"  Part="1"
-AR Path="/5A569D3F/5A559FB3" Ref="R302"  Part="1"
-F 0 "R302" V 3880 5550 50  0000 C CNN
+F 0 "R402" V 3880 5550 50  0000 C CNN
 F 1 "12K" V 3800 5550 50  0000 C CNN
 F 2 "" V 3730 5550 50  0001 C CNN
@@
 $EndComp
 $Comp
-L R R204
+L R R404
 U 1 1 5A55A014
 P 4550 6850
-AR Path="/5A50EA77/5A55A014" Ref="R204"  Part="1"
-AR Path="/5A569D3F/5A55A014" Ref="R304"  Part="1"
-F 0 "R304" V 4630 6850 50  0000 C CNN
+F 0 "R404" V 4630 6850 50  0000 C CNN
 F 1 "12K" V 4550 6850 50  0000 C CNN
 F 2 "" V 4480 6850 50  0001 C CNN
@@
 $EndComp
 $Comp
-L R R203
+L R R403
 U 1 1 5A55A0AD
 P 3800 6600
-AR Path="/5A50EA77/5A55A0AD" Ref="R203"  Part="1"
-AR Path="/5A569D3F/5A55A0AD" Ref="R303"  Part="1"
-F 0 "R303" V 3880 6600 50  0000 C CNN
+F 0 "R403" V 3880 6600 50  0000 C CNN
 F 1 "1K2" V 3800 6600 50  0000 C CNN
 F 2 "" V 3730 6600 50  0001 C CNN
@@
 Connection ~ 4550 6600
 $Comp
-L GND #PWR202
+L GND #PWR402
 U 1 1 5A55A389
 P 4750 7000
-AR Path="/5A50EA77/5A55A389" Ref="#PWR202"  Part="1"
-AR Path="/5A569D3F/5A55A389" Ref="#PWR302"  Part="1"
-F 0 "#PWR302" H 4750 6750 50  0001 C CNN
+F 0 "#PWR402" H 4750 6750 50  0001 C CNN
 F 1 "GND" H 4750 6850 50  0000 C CNN
 F 2 "" H 4750 7000 50  0001 C CNN
@@
 Connection ~ 4750 7000
 $Comp
-L R R201
-U 1 1 5A55A50D
+L R R401
+U 1 1 5A57FC94
 P 3500 6350
-AR Path="/5A50EA77/5A55A50D" Ref="R201"  Part="1"
-AR Path="/5A569D3F/5A55A50D" Ref="R301"  Part="1"
-F 0 "R301" V 3580 6350 50  0000 C CNN
+F 0 "R401" V 3580 6350 50  0000 C CNN
 F 1 "22" V 3500 6350 50  0000 C CNN
 F 2 "" V 3430 6350 50  0001 C CNN
@@
 	9650 1050 9350 1050
 $Comp
-L Jumper_NC_Small JP202
+L Jumper_NC_Small JP402
 U 1 1 5A55DB5B
 P 9450 1200
-AR Path="/5A50EA77/5A55DB5B" Ref="JP202"  Part="1"
-AR Path="/5A569D3F/5A55DB5B" Ref="JP302"  Part="1"
-F 0 "JP302" H 9450 1280 50  0000 C CNN
+F 0 "JP402" H 9450 1280 50  0000 C CNN
 F 1 "Jmp" H 9460 1140 50  0000 C CNN
 F 2 "" H 9450 1200 50  0001 C CNN
