File: Electrical/Common/Stepper.sch (KiCad schematic (older format))
At the start: 12 parts, among them Q401 FDC6420C

Commit message: Completed quad schematics
Parts:
- renumbered A401 to A301, A402 to A302, A403 to A303, A404 to A304, JP401 to JP301, JP402 to JP302, JP403 to JP303, Q401 to Q301, R401 to R301, R402 to R302, R403 to R303, R404 to R304
Changed lines of the file:
@@
 LIBS:dc-dc
 LIBS:allegro
-LIBS:Dual-cache
+LIBS:Quad-cache
 EELAYER 25 0
 EELAYER END
 $Descr A4 11693 8268
 encoding utf-8
-Sheet 4 4
+Sheet 3 6
 Title ""
 Date ""
@@
 $EndDescr
 $Comp
-L Pololu_Breakout_A4988 A401
+L Pololu_Breakout_A4988 A301
 U 1 1 5A50EABF
 P 2750 3450
-F 0 "A401" H 2650 4200 50  0000 R CNN
+AR Path="/5A579457/5A50EA77/5A50EABF" Ref="A301"  Part="1"
+AR Path="/5A579457/5A569D3F/5A50EABF" Ref="A401"  Part="1"
+AR Path="/5A5956FB/5A50EABF" Ref="A501"  Part="1"
+AR Path="/5A597FFD/5A50EABF" Ref="A601"  Part="1"
+F 0 "A301" H 2650 4200 50  0000 R CNN
 F 1 "Pololu_Breakout_A4988" H 2650 4100 50  0000 R CNN
 F 2 "Modules:Pololu_Breakout-16_15.2x20.3mm" H 3025 2700 50  0001 L CNN
@@
 $EndComp
 $Comp
-L Pololu_Breakout_DRV8825 A402
+L Pololu_Breakout_DRV8825 A302
 U 1 1 5A50EB28
 P 4750 3400
-F 0 "A402" H 4650 4050 50  0000 R CNN
+AR Path="/5A579457/5A50EA77/5A50EB28" Ref="A302"  Part="1"
+AR Path="/5A579457/5A569D3F/5A50EB28" Ref="A402"  Part="1"
+AR Path="/5A5956FB/5A50EB28" Ref="A502"  Part="1"
+AR Path="/5A597FFD/5A50EB28" Ref="A602"  Part="1"
+F 0 "A302" H 4650 4050 50  0000 R CNN
 F 1 "Pololu_Breakout_DRV8825" H 4650 3950 50  0000 R CNN
 F 2 "Modules:Pololu_Breakout-16_15.2x20.3mm" H 4950 2600 50  0001 L CNN
@@
 $EndComp
 $Comp
-L Pololu_Breakout_DRV8834 A403
+L Pololu_Breakout_DRV8834 A303
 U 1 1 5A50F831
 P 6750 3500
-F 0 "A403" H 6650 4350 50  0000 R CNN
+AR Path="/5A579457/5A50EA77/5A50F831" Ref="A303"  Part="1"
+AR Path="/5A579457/5A569D3F/5A50F831" Ref="A403"  Part="1"
+AR Path="/5A5956FB/5A50F831" Ref="A503"  Part="1"
+AR Path="/5A597FFD/5A50F831" Ref="A603"  Part="1"
+F 0 "A303" H 6650 4350 50  0000 R CNN
 F 1 "Pololu_Breakout_DRV8834" H 6650 4250 50  0000 R CNN
 F 2 "Modules:Pololu_Breakout-16_15.2x20.3mm" H 6950 2700 50  0001 L CNN
@@
 $EndComp
 $Comp
-L Pololu_Breakout_DRV8880 A404
+L Pololu_Breakout_DRV8880 A304
 U 1 1 5A50F8CE
 P 8700 3500
-F 0 "A404" H 8600 4350 50  0000 R CNN
+AR Path="/5A579457/5A50EA77/5A50F8CE" Ref="A304"  Part="1"
+AR Path="/5A579457/5A569D3F/5A50F8CE" Ref="A404"  Part="1"
+AR Path="/5A5956FB/5A50F8CE" Ref="A504"  Part="1"
+AR Path="/5A597FFD/5A50F8CE" Ref="A604"  Part="1"
+F 0 "A304" H 8600 4350 50  0000 R CNN
 F 1 "Pololu_Breakout_DRV8880" H 8600 4250 50  0000 R CNN
 F 2 "Modules:Pololu_Breakout-16_15.2x20.3mm" H 8900 2700 50  0001 L CNN
@@
 DIR
 $Comp
-L GND #PWR405
+L GND #PWR305
 U 1 1 5A50FF78
 P 8800 4350
-F 0 "#PWR405" H 8800 4100 50  0001 C CNN
+AR Path="/5A579457/5A50EA77/5A50FF78" Ref="#PWR305"  Part="1"
+AR Path="/5A579457/5A569D3F/5A50FF78" Ref="#PWR405"  Part="1"
+AR Path="/5A5956FB/5A50FF78" Ref="#PWR505"  Part="1"
+AR Path="/5A597FFD/5A50FF78" Ref="#PWR605"  Part="1"
+F 0 "#PWR305" H 8800 4100 50  0001 C CNN
 F 1 "GND" H 8800 4200 50  0000 C CNN
 F 2 "" H 8800 4350 50  0001 C CNN
@@
 	8800 4300 8700 4300
 $Comp
-L GND #PWR404
+L GND #PWR304
 U 1 1 5A50FFB9
 P 6950 4350
-F 0 "#PWR404" H 6950 4100 50  0001 C CNN
+AR Path="/5A579457/5A50EA77/5A50FFB9" Ref="#PWR304"  Part="1"
+AR Path="/5A579457/5A569D3F/5A50FFB9" Ref="#PWR404"  Part="1"
+AR Path="/5A5956FB/5A50FFB9" Ref="#PWR504"  Part="1"
+AR Path="/5A597FFD/5A50FFB9" Ref="#PWR604"  Part="1"
+F 0 "#PWR304" H 6950 4100 50  0001 C CNN
 F 1 "GND" H 6950 4200 50  0000 C CNN
 F 2 "" H 6950 4350 50  0001 C CNN
@@
 $EndComp
 $Comp
-L GND #PWR403
+L GND #PWR303
 U 1 1 5A50FFD0
 P 4850 4250
-F 0 "#PWR403" H 4850 4000 50  0001 C CNN
+AR Path="/5A579457/5A50EA77/5A50FFD0" Ref="#PWR303"  Part="1"
+AR Path="/5A579457/5A569D3F/5A50FFD0" Ref="#PWR403"  Part="1"
+AR Path="/5A5956FB/5A50FFD0" Ref="#PWR503"  Part="1"
+AR Path="/5A597FFD/5A50FFD0" Ref="#PWR603"  Part="1"
+F 0 "#PWR303" H 4850 4000 50  0001 C CNN
 F 1 "GND" H 4850 4100 50  0000 C CNN
 F 2 "" H 4850 4250 50  0001 C CNN
@@
 $EndComp
 $Comp
-L GND #PWR401
+L GND #PWR301
 U 1 1 5A57FC8B
 P 2950 4300
-F 0 "#PWR401" H 2950 4050 50  0001 C CNN
+AR Path="/5A579457/5A50EA77/5A57FC8B" Ref="#PWR301"  Part="1"
+AR Path="/5A579457/5A569D3F/5A57FC8B" Ref="#PWR401"  Part="1"
+AR Path="/5A5956FB/5A57FC8B" Ref="#PWR501"  Part="1"
+AR Path="/5A597FFD/5A57FC8B" Ref="#PWR601"  Part="1"
+F 0 "#PWR301" H 2950 4050 50  0001 C CNN
 F 1 "GND" H 2950 4150 50  0000 C CNN
 F 2 "" H 2950 4300 50  0001 C CNN
@@
 Vadj
 $Comp
-L Conn_01x03 JP401
+L Conn_01x03 JP301
 U 1 1 5A57FC8C
 P 1850 1150
-F 0 "JP401" H 1850 1350 50  0000 C CNN
+AR Path="/5A579457/5A50EA77/5A57FC8C" Ref="JP301"  Part="1"
+AR Path="/5A579457/5A569D3F/5A57FC8C" Ref="JP401"  Part="1"
+AR Path="/5A5956FB/5A57FC8C" Ref="JP501"  Part="1"
+AR Path="/5A597FFD/5A57FC8C" Ref="JP601"  Part="1"
+F 0 "JP301" H 1850 1350 50  0000 C CNN
 F 1 "01x03" H 1850 950 50  0000 C CNN
 F 2 "" H 1850 1150 50  0001 C CNN
@@
 Cfg2
 $Comp
-L Conn_01x02 JP403
+L Conn_01x02 JP303
 U 1 1 5A57FC8D
 P 9850 1050
-F 0 "JP403" H 9850 1150 50  0000 C CNN
+AR Path="/5A579457/5A50EA77/5A57FC8D" Ref="JP303"  Part="1"
+AR Path="/5A579457/5A569D3F/5A57FC8D" Ref="JP403"  Part="1"
+AR Path="/5A5956FB/5A57FC8D" Ref="JP503"  Part="1"
+AR Path="/5A597FFD/5A57FC8D" Ref="JP603"  Part="1"
+F 0 "JP303" H 9850 1150 50  0000 C CNN
 F 1 "01x02" H 9850 850 50  0000 C CNN
 F 2 "" H 9850 1050 50  0001 C CNN
@@
 SLP
 $Comp
-L FDC6420C Q401
+L FDC6420C Q301
 U 2 1 5A57FC8E
 P 4750 6650
-F 0 "Q401" H 4950 6725 50  0000 L CNN
+AR Path="/5A579457/5A50EA77/5A57FC8E" Ref="Q301"  Part="2"
+AR Path="/5A579457/5A569D3F/5A57FC8E" Ref="Q401"  Part="2"
+AR Path="/5A5956FB/5A57FC8E" Ref="Q501"  Part="2"
+AR Path="/5A597FFD/5A57FC8E" Ref="Q601"  Part="2"
+F 0 "Q301" H 4950 6725 50  0000 L CNN
 F 1 "FDC6420C" H 4950 6650 50  0000 L CNN
 F 2 "TO_SOT_Packages_SMD:SOT-363_SC-70-6" H 4950 6575 50  0001 L CIN
@@
 $EndComp
 $Comp
-L FDC6420C Q401
+L FDC6420C Q301
 U 1 1 5A57FC8F
 P 3600 5950
-F 0 "Q401" H 3800 6025 50  0000 L CNN
+AR Path="/5A579457/5A50EA77/5A57FC8F" Ref="Q301"  Part="1"
+AR Path="/5A579457/5A569D3F/5A57FC8F" Ref="Q401"  Part="1"
+AR Path="/5A5956FB/5A57FC8F" Ref="Q501"  Part="1"
+AR Path="/5A597FFD/5A57FC8F" Ref="Q601"  Part="1"
+F 0 "Q301" H 3800 6025 50  0000 L CNN
 F 1 "FDC6420C" H 3800 5950 50  0000 L CNN
 F 2 "TO_SOT_Packages_SMD:SOT-363_SC-70-6" H 3800 5875 50  0001 L CIN
@@
 $EndComp
 $Comp
-L R R402
+L R R302
 U 1 1 5A559FB3
 P 3800 5550
-F 0 "R402" V 3880 5550 50  0000 C CNN
+AR Path="/5A579457/5A50EA77/5A559FB3" Ref="R302"  Part="1"
+AR Path="/5A579457/5A569D3F/5A559FB3" Ref="R402"  Part="1"
+AR Path="/5A5956FB/5A559FB3" Ref="R502"  Part="1"
+AR Path="/5A597FFD/5A559FB3" Ref="R602"  Part="1"
+F 0 "R302" V 3880 5550 50  0000 C CNN
 F 1 "12K" V 3800 5550 50  0000 C CNN
 F 2 "" V 3730 5550 50  0001 C CNN
@@
 $EndComp
 $Comp
-L R R404
+L R R304
 U 1 1 5A55A014
 P 4550 6850
-F 0 "R404" V 4630 6850 50  0000 C CNN
+AR Path="/5A579457/5A50EA77/5A55A014" Ref="R304"  Part="1"
+AR Path="/5A579457/5A569D3F/5A55A014" Ref="R404"  Part="1"
+AR Path="/5A5956FB/5A55A014" Ref="R504"  Part="1"
+AR Path="/5A597FFD/5A55A014" Ref="R604"  Part="1"
+F 0 "R304" V 4630 6850 50  0000 C CNN
 F 1 "12K" V 4550 6850 50  0000 C CNN
 F 2 "" V 4480 6850 50  0001 C CNN
@@
 $EndComp
 $Comp
-L R R403
+L R R303
 U 1 1 5A55A0AD
 P 3800 6600
-F 0 "R403" V 3880 6600 50  0000 C CNN
+AR Path="/5A579457/5A50EA77/5A55A0AD" Ref="R303"  Part="1"
+AR Path="/5A579457/5A569D3F/5A55A0AD" Ref="R403"  Part="1"
+AR Path="/5A5956FB/5A55A0AD" Ref="R503"  Part="1"
+AR Path="/5A597FFD/5A55A0AD" Ref="R603"  Part="1"
+F 0 "R303" V 3880 6600 50  0000 C CNN
 F 1 "1K2" V 3800 6600 50  0000 C CNN
 F 2 "" V 3730 6600 50  0001 C CNN
@@
 Connection ~ 4550 6600
 $Comp
-L GND #PWR402
+L GND #PWR302
 U 1 1 5A55A389
 P 4750 7000
-F 0 "#PWR402" H 4750 6750 50  0001 C CNN
+AR Path="/5A579457/5A50EA77/5A55A389" Ref="#PWR302"  Part="1"
+AR Path="/5A579457/5A569D3F/5A55A389" Ref="#PWR402"  Part="1"
+AR Path="/5A5956FB/5A55A389" Ref="#PWR502"  Part="1"
+AR Path="/5A597FFD/5A55A389" Ref="#PWR602"  Part="1"
+F 0 "#PWR302" H 4750 6750 50  0001 C CNN
 F 1 "GND" H 4750 6850 50  0000 C CNN
 F 2 "" H 4750 7000 50  0001 C CNN
@@
 Connection ~ 4750 7000
 $Comp
-L R R401
+L R R301
 U 1 1 5A57FC94
 P 3500 6350
-F 0 "R401" V 3580 6350 50  0000 C CNN
+AR Path="/5A579457/5A50EA77/5A57FC94" Ref="R301"  Part="1"
+AR Path="/5A579457/5A569D3F/5A57FC94" Ref="R401"  Part="1"
+AR Path="/5A5956FB/5A57FC94" Ref="R501"  Part="1"
+AR Path="/5A597FFD/5A57FC94" Ref="R601"  Part="1"
+F 0 "R301" V 3580 6350 50  0000 C CNN
 F 1 "22" V 3500 6350 50  0000 C CNN
 F 2 "" V 3430 6350 50  0001 C CNN
@@
 	9650 1050 9350 1050
 $Comp
-L Jumper_NC_Small JP402
+L Jumper_NC_Small JP302
 U 1 1 5A55DB5B
 P 9450 1200
-F 0 "JP402" H 9450 1280 50  0000 C CNN
+AR Path="/5A579457/5A50EA77/5A55DB5B" Ref="JP302"  Part="1"
+AR Path="/5A579457/5A569D3F/5A55DB5B" Ref="JP402"  Part="1"
+AR Path="/5A5956FB/5A55DB5B" Ref="JP502"  Part="1"
+AR Path="/5A597FFD/5A55DB5B" Ref="JP602"  Part="1"
+F 0 "JP302" H 9450 1280 50  0000 C CNN
 F 1 "Jmp" H 9460 1140 50  0000 C CNN
 F 2 "" H 9450 1200 50  0001 C CNN

Commit message: Fixed DRC errors
Connections:
- net Cfg0: now also A304.10 (M1)
- net Cfg1: now also A304.11 (M0)
- net Cfg2: now also A304.12 (T1)
- net GND: now also A303.1 (GND), A303.7 (GND)
Changed lines of the file:
@@
 LIBS:dc-dc
 LIBS:allegro
-LIBS:Quad-cache
+LIBS:Dual-cache
 EELAYER 25 0
 EELAYER END
 $Descr A4 11693 8268
 encoding utf-8
-Sheet 3 6
+Sheet 3 4
 Title ""
 Date ""
@@
 DIR
 $Comp
-L GND #PWR305
+L GND #PWR039
 U 1 1 5A50FF78
 P 8800 4350
-AR Path="/5A579457/5A50EA77/5A50FF78" Ref="#PWR305"  Part="1"
-AR Path="/5A579457/5A569D3F/5A50FF78" Ref="#PWR405"  Part="1"
-AR Path="/5A5956FB/5A50FF78" Ref="#PWR505"  Part="1"
-AR Path="/5A597FFD/5A50FF78" Ref="#PWR605"  Part="1"
-F 0 "#PWR305" H 8800 4100 50  0001 C CNN
+AR Path="/5A579457/5A50EA77/5A50FF78" Ref="#PWR039"  Part="1"
+AR Path="/5A579457/5A569D3F/5A50FF78" Ref="#PWR045"  Part="1"
+AR Path="/5A5956FB/5A50FF78" Ref="#PWR051"  Part="1"
+AR Path="/5A597FFD/5A50FF78" Ref="#PWR057"  Part="1"
+F 0 "#PWR045" H 8800 4100 50  0001 C CNN
 F 1 "GND" H 8800 4200 50  0000 C CNN
 F 2 "" H 8800 4350 50  0001 C CNN
@@
 	8800 4300 8700 4300
 $Comp
-L GND #PWR304
+L GND #PWR040
 U 1 1 5A50FFB9
 P 6950 4350
-AR Path="/5A579457/5A50EA77/5A50FFB9" Ref="#PWR304"  Part="1"
-AR Path="/5A579457/5A569D3F/5A50FFB9" Ref="#PWR404"  Part="1"
-AR Path="/5A5956FB/5A50FFB9" Ref="#PWR504"  Part="1"
-AR Path="/5A597FFD/5A50FFB9" Ref="#PWR604"  Part="1"
-F 0 "#PWR304" H 6950 4100 50  0001 C CNN
+AR Path="/5A579457/5A50EA77/5A50FFB9" Ref="#PWR040"  Part="1"
+AR Path="/5A579457/5A569D3F/5A50FFB9" Ref="#PWR046"  Part="1"
+AR Path="/5A5956FB/5A50FFB9" Ref="#PWR052"  Part="1"
+AR Path="/5A597FFD/5A50FFB9" Ref="#PWR058"  Part="1"
+F 0 "#PWR046" H 6950 4100 50  0001 C CNN
 F 1 "GND" H 6950 4200 50  0000 C CNN
 F 2 "" H 6950 4350 50  0001 C CNN
@@
 $EndComp
 $Comp
-L GND #PWR303
+L GND #PWR041
 U 1 1 5A50FFD0
 P 4850 4250
-AR Path="/5A579457/5A50EA77/5A50FFD0" Ref="#PWR303"  Part="1"
-AR Path="/5A579457/5A569D3F/5A50FFD0" Ref="#PWR403"  Part="1"
-AR Path="/5A5956FB/5A50FFD0" Ref="#PWR503"  Part="1"
-AR Path="/5A597FFD/5A50FFD0" Ref="#PWR603"  Part="1"
-F 0 "#PWR303" H 4850 4000 50  0001 C CNN
+AR Path="/5A579457/5A50EA77/5A50FFD0" Ref="#PWR041"  Part="1"
+AR Path="/5A579457/5A569D3F/5A50FFD0" Ref="#PWR047"  Part="1"
+AR Path="/5A5956FB/5A50FFD0" Ref="#PWR053"  Part="1"
+AR Path="/5A597FFD/5A50FFD0" Ref="#PWR059"  Part="1"
+F 0 "#PWR047" H 4850 4000 50  0001 C CNN
 F 1 "GND" H 4850 4100 50  0000 C CNN
 F 2 "" H 4850 4250 50  0001 C CNN
@@
 $EndComp
 $Comp
-L GND #PWR301
+L GND #PWR042
 U 1 1 5A57FC8B
 P 2950 4300
-AR Path="/5A579457/5A50EA77/5A57FC8B" Ref="#PWR301"  Part="1"
-AR Path="/5A579457/5A569D3F/5A57FC8B" Ref="#PWR401"  Part="1"
-AR Path="/5A5956FB/5A57FC8B" Ref="#PWR501"  Part="1"
-AR Path="/5A597FFD/5A57FC8B" Ref="#PWR601"  Part="1"
-F 0 "#PWR301" H 2950 4050 50  0001 C CNN
+AR Path="/5A579457/5A50EA77/5A57FC8B" Ref="#PWR042"  Part="1"
+AR Path="/5A579457/5A569D3F/5A57FC8B" Ref="#PWR048"  Part="1"
+AR Path="/5A5956FB/5A57FC8B" Ref="#PWR054"  Part="1"
+AR Path="/5A597FFD/5A57FC8B" Ref="#PWR060"  Part="1"
+F 0 "#PWR048" H 2950 4050 50  0001 C CNN
 F 1 "GND" H 2950 4150 50  0000 C CNN
 F 2 "" H 2950 4300 50  0001 C CNN
@@
 Wire Wire Line
 	4850 4200 4750 4200
-Text Label 1650 1150 2    60   ~ 0
+Text Label 1200 1150 2    60   ~ 0
 Vmot
 Text GLabel 1650 950  0    60   Input ~ 0
@@
 Text HLabel 6350 3900 0    60   Input ~ 0
 Cfg1
-Text HLabel 6350 4000 0    60   Input ~ 0
+Text HLabel 8300 4100 0    60   Input ~ 0
 Cfg2
 Text HLabel 6350 3150 0    60   Input ~ 0
@@
 Connection ~ 4550 6600
 $Comp
-L GND #PWR302
+L GND #PWR043
 U 1 1 5A55A389
 P 4750 7000
-AR Path="/5A579457/5A50EA77/5A55A389" Ref="#PWR302"  Part="1"
-AR Path="/5A579457/5A569D3F/5A55A389" Ref="#PWR402"  Part="1"
-AR Path="/5A5956FB/5A55A389" Ref="#PWR502"  Part="1"
-AR Path="/5A597FFD/5A55A389" Ref="#PWR602"  Part="1"
-F 0 "#PWR302" H 4750 6750 50  0001 C CNN
+AR Path="/5A579457/5A50EA77/5A55A389" Ref="#PWR043"  Part="1"
+AR Path="/5A579457/5A569D3F/5A55A389" Ref="#PWR049"  Part="1"
+AR Path="/5A5956FB/5A55A389" Ref="#PWR055"  Part="1"
+AR Path="/5A597FFD/5A55A389" Ref="#PWR061"  Part="1"
+F 0 "#PWR049" H 4750 6750 50  0001 C CNN
 F 1 "GND" H 4750 6850 50  0000 C CNN
 F 2 "" H 4750 7000 50  0001 C CNN
@@
 Text HLabel 4550 6400 1    60   Output ~ 0
 ~FLT
+Wire Wire Line
+	6950 4350 6950 4300
+Wire Wire Line
+	6950 4300 6850 4300
+Text HLabel 8300 3600 0    60   Input ~ 0
+Cfg1
+Text HLabel 8300 3700 0    60   Input ~ 0
+Cfg0
+$Comp
+L PWR_FLAG #FLG044
+U 1 1 5A59046B
+P 1250 1150
+AR Path="/5A579457/5A50EA77/5A59046B" Ref="#FLG044"  Part="1"
+AR Path="/5A579457/5A569D3F/5A59046B" Ref="#FLG050"  Part="1"
+AR Path="/5A5956FB/5A59046B" Ref="#FLG056"  Part="1"
+AR Path="/5A597FFD/5A59046B" Ref="#FLG062"  Part="1"
+F 0 "#FLG050" H 1250 1225 50  0001 C CNN
+F 1 "PWR_FLAG" H 1250 1300 50  0000 C CNN
+F 2 "" H 1250 1150 50  0001 C CNN
+F 3 "" H 1250 1150 50  0001 C CNN
+	1    1250 1150
+	1    0    0    -1
+$EndComp
+Wire Wire Line
+	1200 1150 1650 1150
+Connection ~ 1250 1150
 $EndSCHEMATC

Commit message: Associated footprints. Added some footprint libraries to support.
Parts:
- A304: footprint Modules:Pololu_Breakout-16_15.2x20.3mm -> footprints:Pololu_Breakout-17_15.2x20.3mm
- JP301: footprint (none) -> Socket_Strips:Socket_Strip_Straight_1x03_Pitch2.54mm
- JP302: value Jmp -> JPNC; footprint (none) -> footprints:JPNC
- JP303: footprint (none) -> Socket_Strips:Socket_Strip_Straight_1x02_Pitch2.54mm
- R301, R302, R303, R304: footprint (none) -> Resistors_SMD:R_0603_HandSoldering
Changed lines of the file:
@@
 AR Path="/5A5956FB/5A50EABF" Ref="A501"  Part="1"
 AR Path="/5A597FFD/5A50EABF" Ref="A601"  Part="1"
-F 0 "A301" H 2650 4200 50  0000 R CNN
+F 0 "A401" H 2650 4200 50  0000 R CNN
 F 1 "Pololu_Breakout_A4988" H 2650 4100 50  0000 R CNN
 F 2 "Modules:Pololu_Breakout-16_15.2x20.3mm" H 3025 2700 50  0001 L CNN
@@
 AR Path="/5A5956FB/5A50EB28" Ref="A502"  Part="1"
 AR Path="/5A597FFD/5A50EB28" Ref="A602"  Part="1"
-F 0 "A302" H 4650 4050 50  0000 R CNN
+F 0 "A402" H 4650 4050 50  0000 R CNN
 F 1 "Pololu_Breakout_DRV8825" H 4650 3950 50  0000 R CNN
 F 2 "Modules:Pololu_Breakout-16_15.2x20.3mm" H 4950 2600 50  0001 L CNN
@@
 AR Path="/5A5956FB/5A50F831" Ref="A503"  Part="1"
 AR Path="/5A597FFD/5A50F831" Ref="A603"  Part="1"
-F 0 "A303" H 6650 4350 50  0000 R CNN
+F 0 "A403" H 6650 4350 50  0000 R CNN
 F 1 "Pololu_Breakout_DRV8834" H 6650 4250 50  0000 R CNN
 F 2 "Modules:Pololu_Breakout-16_15.2x20.3mm" H 6950 2700 50  0001 L CNN
@@
 AR Path="/5A5956FB/5A50F8CE" Ref="A504"  Part="1"
 AR Path="/5A597FFD/5A50F8CE" Ref="A604"  Part="1"
-F 0 "A304" H 8600 4350 50  0000 R CNN
+F 0 "A404" H 8600 4350 50  0000 R CNN
 F 1 "Pololu_Breakout_DRV8880" H 8600 4250 50  0000 R CNN
-F 2 "Modules:Pololu_Breakout-16_15.2x20.3mm" H 8900 2700 50  0001 L CNN
+F 2 "footprints:Pololu_Breakout-17_15.2x20.3mm" H 8900 2700 50  0001 L CNN
 F 3 "" H 8800 3200 50  0001 C CNN
 	1    8700 3500
@@
 AR Path="/5A5956FB/5A57FC8C" Ref="JP501"  Part="1"
 AR Path="/5A597FFD/5A57FC8C" Ref="JP601"  Part="1"
-F 0 "JP301" H 1850 1350 50  0000 C CNN
+F 0 "JP401" H 1850 1350 50  0000 C CNN
 F 1 "01x03" H 1850 950 50  0000 C CNN
-F 2 "" H 1850 1150 50  0001 C CNN
+F 2 "Socket_Strips:Socket_Strip_Straight_1x03_Pitch2.54mm" H 1850 1150 50  0001 C CNN
 F 3 "" H 1850 1150 50  0001 C CNN
 	1    1850 1150
@@
 AR Path="/5A5956FB/5A57FC8D" Ref="JP503"  Part="1"
 AR Path="/5A597FFD/5A57FC8D" Ref="JP603"  Part="1"
-F 0 "JP303" H 9850 1150 50  0000 C CNN
+F 0 "JP403" H 9850 1150 50  0000 C CNN
 F 1 "01x02" H 9850 850 50  0000 C CNN
-F 2 "" H 9850 1050 50  0001 C CNN
+F 2 "Socket_Strips:Socket_Strip_Straight_1x02_Pitch2.54mm" H 9850 1050 50  0001 C CNN
 F 3 "" H 9850 1050 50  0001 C CNN
 	1    9850 1050
@@
 AR Path="/5A5956FB/5A57FC8E" Ref="Q501"  Part="2"
 AR Path="/5A597FFD/5A57FC8E" Ref="Q601"  Part="2"
-F 0 "Q301" H 4950 6725 50  0000 L CNN
+F 0 "Q401" H 4950 6725 50  0000 L CNN
 F 1 "FDC6420C" H 4950 6650 50  0000 L CNN
 F 2 "TO_SOT_Packages_SMD:SOT-363_SC-70-6" H 4950 6575 50  0001 L CIN
@@
 AR Path="/5A5956FB/5A57FC8F" Ref="Q501"  Part="1"
 AR Path="/5A597FFD/5A57FC8F" Ref="Q601"  Part="1"
-F 0 "Q301" H 3800 6025 50  0000 L CNN
+F 0 "Q401" H 3800 6025 50  0000 L CNN
 F 1 "FDC6420C" H 3800 5950 50  0000 L CNN
 F 2 "TO_SOT_Packages_SMD:SOT-363_SC-70-6" H 3800 5875 50  0001 L CIN
@@
 AR Path="/5A5956FB/5A559FB3" Ref="R502"  Part="1"
 AR Path="/5A597FFD/5A559FB3" Ref="R602"  Part="1"
-F 0 "R302" V 3880 5550 50  0000 C CNN
+F 0 "R402" V 3880 5550 50  0000 C CNN
 F 1 "12K" V 3800 5550 50  0000 C CNN
-F 2 "" V 3730 5550 50  0001 C CNN
+F 2 "Resistors_SMD:R_0603_HandSoldering" V 3730 5550 50  0001 C CNN
 F 3 "" H 3800 5550 50  0001 C CNN
 	1    3800 5550
@@
 AR Path="/5A5956FB/5A55A014" Ref="R504"  Part="1"
 AR Path="/5A597FFD/5A55A014" Ref="R604"  Part="1"
-F 0 "R304" V 4630 6850 50  0000 C CNN
+F 0 "R404" V 4630 6850 50  0000 C CNN
 F 1 "12K" V 4550 6850 50  0000 C CNN
-F 2 "" V 4480 6850 50  0001 C CNN
+F 2 "Resistors_SMD:R_0603_HandSoldering" V 4480 6850 50  0001 C CNN
 F 3 "" H 4550 6850 50  0001 C CNN
 	1    4550 6850
@@
 AR Path="/5A5956FB/5A55A0AD" Ref="R503"  Part="1"
 AR Path="/5A597FFD/5A55A0AD" Ref="R603"  Part="1"
-F 0 "R303" V 3880 6600 50  0000 C CNN
+F 0 "R403" V 3880 6600 50  0000 C CNN
 F 1 "1K2" V 3800 6600 50  0000 C CNN
-F 2 "" V 3730 6600 50  0001 C CNN
+F 2 "Resistors_SMD:R_0603_HandSoldering" V 3730 6600 50  0001 C CNN
 F 3 "" H 3800 6600 50  0001 C CNN
 	1    3800 6600
@@
 AR Path="/5A5956FB/5A57FC94" Ref="R501"  Part="1"
 AR Path="/5A597FFD/5A57FC94" Ref="R601"  Part="1"
-F 0 "R301" V 3580 6350 50  0000 C CNN
+F 0 "R401" V 3580 6350 50  0000 C CNN
 F 1 "22" V 3500 6350 50  0000 C CNN
-F 2 "" V 3430 6350 50  0001 C CNN
+F 2 "Resistors_SMD:R_0603_HandSoldering" V 3430 6350 50  0001 C CNN
 F 3 "" H 3500 6350 50  0001 C CNN
 	1    3500 6350
@@
 AR Path="/5A5956FB/5A55DB5B" Ref="JP502"  Part="1"
 AR Path="/5A597FFD/5A55DB5B" Ref="JP602"  Part="1"
-F 0 "JP302" H 9450 1280 50  0000 C CNN
-F 1 "Jmp" H 9460 1140 50  0000 C CNN
-F 2 "" H 9450 1200 50  0001 C CNN
+F 0 "JP402" H 9450 1280 50  0000 C CNN
+F 1 "JPNC" H 9460 1140 50  0000 C CNN
+F 2 "footprints:JPNC" H 9450 1200 50  0001 C CNN
 F 3 "" H 9450 1200 50  0001 C CNN
 	1    9450 1200

Commit message: Fixed issues with socket strips vs pin headers
Parts:
- JP301: footprint Socket_Strips:Socket_Strip_Straight_1x03_Pitch2.54mm -> Pin_Headers:Pin_Header_Straight_1x03_Pitch2.54mm
- JP303: footprint Socket_Strips:Socket_Strip_Straight_1x02_Pitch2.54mm -> Pin_Headers:Pin_Header_Straight_1x02_Pitch2.54mm
Changed lines of the file:
@@
 F 0 "JP401" H 1850 1350 50  0000 C CNN
 F 1 "01x03" H 1850 950 50  0000 C CNN
-F 2 "Socket_Strips:Socket_Strip_Straight_1x03_Pitch2.54mm" H 1850 1150 50  0001 C CNN
+F 2 "Pin_Headers:Pin_Header_Straight_1x03_Pitch2.54mm" H 1850 1150 50  0001 C CNN
 F 3 "" H 1850 1150 50  0001 C CNN
 	1    1850 1150
@@
 F 0 "JP403" H 9850 1150 50  0000 C CNN
 F 1 "01x02" H 9850 850 50  0000 C CNN
-F 2 "Socket_Strips:Socket_Strip_Straight_1x02_Pitch2.54mm" H 9850 1050 50  0001 C CNN
+F 2 "Pin_Headers:Pin_Header_Straight_1x02_Pitch2.54mm" H 9850 1050 50  0001 C CNN
 F 3 "" H 9850 1050 50  0001 C CNN
 	1    9850 1050
