File: Electrical/Common/Stepper.sch (KiCad schematic (older format))
At the start: 12 parts, among them Q301 FDC6420C

Commit message: Working on layout and routing.
Connections:
- net B1: now also A304.5 (B2); no longer A304.6 (B1)
- net B2: now also A304.6 (B1); no longer A304.5 (B2)
Changed lines of the file:
@@
 LIBS:dc-dc
 LIBS:allegro
-LIBS:Quad-cache
+LIBS:mechanical
+LIBS:Dual-cache
 EELAYER 25 0
 EELAYER END
 $Descr A4 11693 8268
 encoding utf-8
-Sheet 3 6
+Sheet 3 4
 Title ""
 Date ""
@@
 Text HLabel 9100 3400 2    60   Output ~ 0
 A1
+Text HLabel 9100 3700 2    60   Output ~ 0
+B1
 Text HLabel 9100 3600 2    60   Output ~ 0
-B1
-Text HLabel 9100 3700 2    60   Output ~ 0
 B2
 Text HLabel 8300 3200 0    60   Input ~ 0
@@
 DIR
 $Comp
-L GND #PWR039
+L GND #PWR040
 U 1 1 5A50FF78
 P 8800 4350
-AR Path="/5A579457/5A50EA77/5A50FF78" Ref="#PWR039"  Part="1"
-AR Path="/5A579457/5A569D3F/5A50FF78" Ref="#PWR045"  Part="1"
+AR Path="/5A579457/5A50EA77/5A50FF78" Ref="#PWR040"  Part="1"
+AR Path="/5A579457/5A569D3F/5A50FF78" Ref="#PWR046"  Part="1"
 AR Path="/5A5956FB/5A50FF78" Ref="#PWR051"  Part="1"
 AR Path="/5A597FFD/5A50FF78" Ref="#PWR057"  Part="1"
-F 0 "#PWR057" H 8800 4100 50  0001 C CNN
+F 0 "#PWR046" H 8800 4100 50  0001 C CNN
 F 1 "GND" H 8800 4200 50  0000 C CNN
 F 2 "" H 8800 4350 50  0001 C CNN
@@
 	8800 4300 8700 4300
 $Comp
-L GND #PWR040
+L GND #PWR041
 U 1 1 5A50FFB9
 P 6950 4350
-AR Path="/5A579457/5A50EA77/5A50FFB9" Ref="#PWR040"  Part="1"
-AR Path="/5A579457/5A569D3F/5A50FFB9" Ref="#PWR046"  Part="1"
+AR Path="/5A579457/5A50EA77/5A50FFB9" Ref="#PWR041"  Part="1"
+AR Path="/5A579457/5A569D3F/5A50FFB9" Ref="#PWR047"  Part="1"
 AR Path="/5A5956FB/5A50FFB9" Ref="#PWR052"  Part="1"
 AR Path="/5A597FFD/5A50FFB9" Ref="#PWR058"  Part="1"
-F 0 "#PWR058" H 6950 4100 50  0001 C CNN
+F 0 "#PWR047" H 6950 4100 50  0001 C CNN
 F 1 "GND" H 6950 4200 50  0000 C CNN
 F 2 "" H 6950 4350 50  0001 C CNN
@@
 $EndComp
 $Comp
-L GND #PWR041
+L GND #PWR042
 U 1 1 5A50FFD0
 P 4850 4250
-AR Path="/5A579457/5A50EA77/5A50FFD0" Ref="#PWR041"  Part="1"
-AR Path="/5A579457/5A569D3F/5A50FFD0" Ref="#PWR047"  Part="1"
+AR Path="/5A579457/5A50EA77/5A50FFD0" Ref="#PWR042"  Part="1"
+AR Path="/5A579457/5A569D3F/5A50FFD0" Ref="#PWR048"  Part="1"
 AR Path="/5A5956FB/5A50FFD0" Ref="#PWR053"  Part="1"
 AR Path="/5A597FFD/5A50FFD0" Ref="#PWR059"  Part="1"
-F 0 "#PWR059" H 4850 4000 50  0001 C CNN
+F 0 "#PWR048" H 4850 4000 50  0001 C CNN
 F 1 "GND" H 4850 4100 50  0000 C CNN
 F 2 "" H 4850 4250 50  0001 C CNN
@@
 $EndComp
 $Comp
-L GND #PWR042
+L GND #PWR043
 U 1 1 5A57FC8B
 P 2950 4300
-AR Path="/5A579457/5A50EA77/5A57FC8B" Ref="#PWR042"  Part="1"
-AR Path="/5A579457/5A569D3F/5A57FC8B" Ref="#PWR048"  Part="1"
+AR Path="/5A579457/5A50EA77/5A57FC8B" Ref="#PWR043"  Part="1"
+AR Path="/5A579457/5A569D3F/5A57FC8B" Ref="#PWR049"  Part="1"
 AR Path="/5A5956FB/5A57FC8B" Ref="#PWR054"  Part="1"
 AR Path="/5A597FFD/5A57FC8B" Ref="#PWR060"  Part="1"
-F 0 "#PWR060" H 2950 4050 50  0001 C CNN
+F 0 "#PWR049" H 2950 4050 50  0001 C CNN
 F 1 "GND" H 2950 4150 50  0000 C CNN
 F 2 "" H 2950 4300 50  0001 C CNN
@@
 Connection ~ 4550 6600
 $Comp
-L GND #PWR043
+L GND #PWR044
 U 1 1 5A55A389
 P 4750 7000
-AR Path="/5A579457/5A50EA77/5A55A389" Ref="#PWR043"  Part="1"
-AR Path="/5A579457/5A569D3F/5A55A389" Ref="#PWR049"  Part="1"
+AR Path="/5A579457/5A50EA77/5A55A389" Ref="#PWR044"  Part="1"
+AR Path="/5A579457/5A569D3F/5A55A389" Ref="#PWR050"  Part="1"
 AR Path="/5A5956FB/5A55A389" Ref="#PWR055"  Part="1"
 AR Path="/5A597FFD/5A55A389" Ref="#PWR061"  Part="1"
-F 0 "#PWR061" H 4750 6750 50  0001 C CNN
+F 0 "#PWR050" H 4750 6750 50  0001 C CNN
 F 1 "GND" H 4750 6850 50  0000 C CNN
 F 2 "" H 4750 7000 50  0001 C CNN
@@
 Cfg0
 $Comp
-L PWR_FLAG #FLG044
+L PWR_FLAG #FLG045
 U 1 1 5A59046B
 P 1250 1150
-AR Path="/5A579457/5A50EA77/5A59046B" Ref="#FLG044"  Part="1"
-AR Path="/5A579457/5A569D3F/5A59046B" Ref="#FLG050"  Part="1"
+AR Path="/5A579457/5A50EA77/5A59046B" Ref="#FLG045"  Part="1"
+AR Path="/5A579457/5A569D3F/5A59046B" Ref="#FLG051"  Part="1"
 AR Path="/5A5956FB/5A59046B" Ref="#FLG056"  Part="1"
 AR Path="/5A597FFD/5A59046B" Ref="#FLG062"  Part="1"
-F 0 "#FLG062" H 1250 1225 50  0001 C CNN
+F 0 "#FLG051" H 1250 1225 50  0001 C CNN
 F 1 "PWR_FLAG" H 1250 1300 50  0000 C CNN
 F 2 "" H 1250 1150 50  0001 C CNN
