File: Electrical/Common/Stepper.sch (KiCad schematic (older format))
At the start: 12 parts, among them Q301 FDC6420C

Commit message: Added a diode to the stepper fault/3v3 supply to ensure fault remains low when RESET/PMIC_OUT_PGOOD is low.
Parts:
- added D401: D, footprints:D_0603_HandSoldering, symbol D
- A301, A302, A303: footprint Modules:Pololu_Breakout-16_15.2x20.3mm -> footprints:Pololu_Breakout-16_15.2x20.3mm
Connections:
- net labels added: RST
- wire segments 30 -> 31
Changed lines of the file:
@@
 AR Path="/5A5956FB/5A50EABF" Ref="A501"  Part="1"
 AR Path="/5A597FFD/5A50EABF" Ref="A601"  Part="1"
-F 0 "A401" H 2650 4200 50  0000 R CNN
+F 0 "A301" H 2650 4200 50  0000 R CNN
 F 1 "Pololu_Breakout_A4988" H 2650 4100 50  0000 R CNN
-F 2 "Modules:Pololu_Breakout-16_15.2x20.3mm" H 3025 2700 50  0001 L CNN
+F 2 "footprints:Pololu_Breakout-16_15.2x20.3mm" H 3025 2700 50  0001 L CNN
 F 3 "" H 2850 3150 50  0001 C CNN
 	1    2750 3450
@@
 AR Path="/5A5956FB/5A50EB28" Ref="A502"  Part="1"
 AR Path="/5A597FFD/5A50EB28" Ref="A602"  Part="1"
-F 0 "A402" H 4650 4050 50  0000 R CNN
+F 0 "A302" H 4650 4050 50  0000 R CNN
 F 1 "Pololu_Breakout_DRV8825" H 4650 3950 50  0000 R CNN
-F 2 "Modules:Pololu_Breakout-16_15.2x20.3mm" H 4950 2600 50  0001 L CNN
+F 2 "footprints:Pololu_Breakout-16_15.2x20.3mm" H 4950 2600 50  0001 L CNN
 F 3 "" H 4850 3100 50  0001 C CNN
 	1    4750 3400
@@
 AR Path="/5A5956FB/5A50F831" Ref="A503"  Part="1"
 AR Path="/5A597FFD/5A50F831" Ref="A603"  Part="1"
-F 0 "A403" H 6650 4350 50  0000 R CNN
+F 0 "A303" H 6650 4350 50  0000 R CNN
 F 1 "Pololu_Breakout_DRV8834" H 6650 4250 50  0000 R CNN
-F 2 "Modules:Pololu_Breakout-16_15.2x20.3mm" H 6950 2700 50  0001 L CNN
+F 2 "footprints:Pololu_Breakout-16_15.2x20.3mm" H 6950 2700 50  0001 L CNN
 F 3 "" H 6850 3300 50  0001 C CNN
 	1    6750 3500
@@
 AR Path="/5A5956FB/5A50F8CE" Ref="A504"  Part="1"
 AR Path="/5A597FFD/5A50F8CE" Ref="A604"  Part="1"
-F 0 "A404" H 8600 4350 50  0000 R CNN
+F 0 "A304" H 8600 4350 50  0000 R CNN
 F 1 "Pololu_Breakout_DRV8880" H 8600 4250 50  0000 R CNN
 F 2 "footprints:Pololu_Breakout-17_15.2x20.3mm" H 8900 2700 50  0001 L CNN
@@
 DIR
 $Comp
-L GND #PWR041
+L GND #PWR304
 U 1 1 5A50FF78
 P 8800 4350
-AR Path="/5A579457/5A50EA77/5A50FF78" Ref="#PWR041"  Part="1"
-AR Path="/5A579457/5A569D3F/5A50FF78" Ref="#PWR047"  Part="1"
-AR Path="/5A5956FB/5A50FF78" Ref="#PWR051"  Part="1"
-AR Path="/5A597FFD/5A50FF78" Ref="#PWR057"  Part="1"
-F 0 "#PWR047" H 8800 4100 50  0001 C CNN
+AR Path="/5A579457/5A50EA77/5A50FF78" Ref="#PWR304"  Part="1"
+AR Path="/5A579457/5A569D3F/5A50FF78" Ref="#PWR404"  Part="1"
+AR Path="/5A5956FB/5A50FF78" Ref="#PWR052"  Part="1"
+AR Path="/5A597FFD/5A50FF78" Ref="#PWR058"  Part="1"
+F 0 "#PWR304" H 8800 4100 50  0001 C CNN
 F 1 "GND" H 8800 4200 50  0000 C CNN
 F 2 "" H 8800 4350 50  0001 C CNN
@@
 	8800 4300 8700 4300
 $Comp
-L GND #PWR042
+L GND #PWR303
 U 1 1 5A50FFB9
 P 6950 4350
-AR Path="/5A579457/5A50EA77/5A50FFB9" Ref="#PWR042"  Part="1"
-AR Path="/5A579457/5A569D3F/5A50FFB9" Ref="#PWR048"  Part="1"
-AR Path="/5A5956FB/5A50FFB9" Ref="#PWR052"  Part="1"
-AR Path="/5A597FFD/5A50FFB9" Ref="#PWR058"  Part="1"
-F 0 "#PWR048" H 6950 4100 50  0001 C CNN
+AR Path="/5A579457/5A50EA77/5A50FFB9" Ref="#PWR303"  Part="1"
+AR Path="/5A579457/5A569D3F/5A50FFB9" Ref="#PWR403"  Part="1"
+AR Path="/5A5956FB/5A50FFB9" Ref="#PWR053"  Part="1"
+AR Path="/5A597FFD/5A50FFB9" Ref="#PWR059"  Part="1"
+F 0 "#PWR303" H 6950 4100 50  0001 C CNN
 F 1 "GND" H 6950 4200 50  0000 C CNN
 F 2 "" H 6950 4350 50  0001 C CNN
@@
 $EndComp
 $Comp
-L GND #PWR043
+L GND #PWR301
 U 1 1 5A50FFD0
 P 4850 4250
-AR Path="/5A579457/5A50EA77/5A50FFD0" Ref="#PWR043"  Part="1"
-AR Path="/5A579457/5A569D3F/5A50FFD0" Ref="#PWR049"  Part="1"
-AR Path="/5A5956FB/5A50FFD0" Ref="#PWR053"  Part="1"
-AR Path="/5A597FFD/5A50FFD0" Ref="#PWR059"  Part="1"
-F 0 "#PWR049" H 4850 4000 50  0001 C CNN
+AR Path="/5A579457/5A50EA77/5A50FFD0" Ref="#PWR301"  Part="1"
+AR Path="/5A579457/5A569D3F/5A50FFD0" Ref="#PWR401"  Part="1"
+AR Path="/5A5956FB/5A50FFD0" Ref="#PWR054"  Part="1"
+AR Path="/5A597FFD/5A50FFD0" Ref="#PWR060"  Part="1"
+F 0 "#PWR301" H 4850 4000 50  0001 C CNN
 F 1 "GND" H 4850 4100 50  0000 C CNN
 F 2 "" H 4850 4250 50  0001 C CNN
@@
 $EndComp
 $Comp
-L GND #PWR044
+L GND #PWR302
 U 1 1 5A57FC8B
 P 2950 4300
-AR Path="/5A579457/5A50EA77/5A57FC8B" Ref="#PWR044"  Part="1"
-AR Path="/5A579457/5A569D3F/5A57FC8B" Ref="#PWR050"  Part="1"
-AR Path="/5A5956FB/5A57FC8B" Ref="#PWR054"  Part="1"
-AR Path="/5A597FFD/5A57FC8B" Ref="#PWR060"  Part="1"
-F 0 "#PWR050" H 2950 4050 50  0001 C CNN
+AR Path="/5A579457/5A50EA77/5A57FC8B" Ref="#PWR302"  Part="1"
+AR Path="/5A579457/5A569D3F/5A57FC8B" Ref="#PWR402"  Part="1"
+AR Path="/5A5956FB/5A57FC8B" Ref="#PWR055"  Part="1"
+AR Path="/5A597FFD/5A57FC8B" Ref="#PWR061"  Part="1"
+F 0 "#PWR302" H 2950 4050 50  0001 C CNN
 F 1 "GND" H 2950 4150 50  0000 C CNN
 F 2 "" H 2950 4300 50  0001 C CNN
@@
 AR Path="/5A5956FB/5A57FC8C" Ref="JP501"  Part="1"
 AR Path="/5A597FFD/5A57FC8C" Ref="JP601"  Part="1"
-F 0 "JP401" H 1850 1350 50  0000 C CNN
+F 0 "JP301" H 1850 1350 50  0000 C CNN
 F 1 "01x03" H 1850 950 50  0000 C CNN
 F 2 "Pin_Headers:Pin_Header_Straight_1x03_Pitch2.54mm" H 1850 1150 50  0001 C CNN
@@
 AR Path="/5A5956FB/5A57FC8D" Ref="JP503"  Part="1"
 AR Path="/5A597FFD/5A57FC8D" Ref="JP603"  Part="1"
-F 0 "JP403" H 9850 1150 50  0000 C CNN
+F 0 "JP303" H 9850 1150 50  0000 C CNN
 F 1 "01x02" H 9850 850 50  0000 C CNN
 F 2 "Pin_Headers:Pin_Header_Straight_1x02_Pitch2.54mm" H 9850 1050 50  0001 C CNN
@@
 AR Path="/5A5956FB/5A57FC8E" Ref="Q501"  Part="2"
 AR Path="/5A597FFD/5A57FC8E" Ref="Q601"  Part="2"
-F 0 "Q401" H 4950 6725 50  0000 L CNN
+F 0 "Q301" H 4950 6725 50  0000 L CNN
 F 1 "FDC6420C" H 4950 6650 50  0000 L CNN
 F 2 "TO_SOT_Packages_SMD:SOT-363_SC-70-6" H 4950 6575 50  0001 L CIN
@@
 AR Path="/5A5956FB/5A57FC8F" Ref="Q501"  Part="1"
 AR Path="/5A597FFD/5A57FC8F" Ref="Q601"  Part="1"
-F 0 "Q401" H 3800 6025 50  0000 L CNN
+F 0 "Q301" H 3800 6025 50  0000 L CNN
 F 1 "FDC6420C" H 3800 5950 50  0000 L CNN
 F 2 "TO_SOT_Packages_SMD:SOT-363_SC-70-6" H 3800 5875 50  0001 L CIN
@@
 AR Path="/5A5956FB/5A559FB3" Ref="R502"  Part="1"
 AR Path="/5A597FFD/5A559FB3" Ref="R602"  Part="1"
-F 0 "R402" V 3880 5550 50  0000 C CNN
+F 0 "R302" V 3880 5550 50  0000 C CNN
 F 1 "12K" V 3800 5550 50  0000 C CNN
 F 2 "Resistors_SMD:R_0603_HandSoldering" V 3730 5550 50  0001 C CNN
@@
 AR Path="/5A5956FB/5A55A014" Ref="R504"  Part="1"
 AR Path="/5A597FFD/5A55A014" Ref="R604"  Part="1"
-F 0 "R404" V 4630 6850 50  0000 C CNN
+F 0 "R304" V 4630 6850 50  0000 C CNN
 F 1 "12K" V 4550 6850 50  0000 C CNN
 F 2 "Resistors_SMD:R_0603_HandSoldering" V 4480 6850 50  0001 C CNN
@@
 AR Path="/5A5956FB/5A55A0AD" Ref="R503"  Part="1"
 AR Path="/5A597FFD/5A55A0AD" Ref="R603"  Part="1"
-F 0 "R403" V 3880 6600 50  0000 C CNN
+F 0 "R303" V 3880 6600 50  0000 C CNN
 F 1 "1K2" V 3800 6600 50  0000 C CNN
 F 2 "Resistors_SMD:R_0603_HandSoldering" V 3730 6600 50  0001 C CNN
@@
 Connection ~ 4550 6600
 $Comp
-L GND #PWR045
+L GND #PWR305
 U 1 1 5A55A389
 P 4750 7000
-AR Path="/5A579457/5A50EA77/5A55A389" Ref="#PWR045"  Part="1"
-AR Path="/5A579457/5A569D3F/5A55A389" Ref="#PWR051"  Part="1"
-AR Path="/5A5956FB/5A55A389" Ref="#PWR055"  Part="1"
-AR Path="/5A597FFD/5A55A389" Ref="#PWR061"  Part="1"
-F 0 "#PWR051" H 4750 6750 50  0001 C CNN
+AR Path="/5A579457/5A50EA77/5A55A389" Ref="#PWR305"  Part="1"
+AR Path="/5A579457/5A569D3F/5A55A389" Ref="#PWR405"  Part="1"
+AR Path="/5A5956FB/5A55A389" Ref="#PWR056"  Part="1"
+AR Path="/5A597FFD/5A55A389" Ref="#PWR062"  Part="1"
+F 0 "#PWR305" H 4750 6750 50  0001 C CNN
 F 1 "GND" H 4750 6850 50  0000 C CNN
 F 2 "" H 4750 7000 50  0001 C CNN
@@
 AR Path="/5A5956FB/5A57FC94" Ref="R501"  Part="1"
 AR Path="/5A597FFD/5A57FC94" Ref="R601"  Part="1"
-F 0 "R401" V 3580 6350 50  0000 C CNN
+F 0 "R301" V 3580 6350 50  0000 C CNN
 F 1 "22" V 3500 6350 50  0000 C CNN
 F 2 "Resistors_SMD:R_0603_HandSoldering" V 3430 6350 50  0001 C CNN
@@
 AR Path="/5A5956FB/5A55DB5B" Ref="JP502"  Part="1"
 AR Path="/5A597FFD/5A55DB5B" Ref="JP602"  Part="1"
-F 0 "JP402" H 9450 1280 50  0000 C CNN
+F 0 "JP302" H 9450 1280 50  0000 C CNN
 F 1 "JPNC" H 9460 1140 50  0000 C CNN
 F 2 "footprints:JPNC" H 9450 1200 50  0001 C CNN
@@
 Cfg0
 $Comp
-L PWR_FLAG #FLG046
+L PWR_FLAG #FLG301
 U 1 1 5A59046B
 P 1250 1150
-AR Path="/5A579457/5A50EA77/5A59046B" Ref="#FLG046"  Part="1"
-AR Path="/5A579457/5A569D3F/5A59046B" Ref="#FLG052"  Part="1"
-AR Path="/5A5956FB/5A59046B" Ref="#FLG056"  Part="1"
-AR Path="/5A597FFD/5A59046B" Ref="#FLG062"  Part="1"
-F 0 "#FLG052" H 1250 1225 50  0001 C CNN
+AR Path="/5A579457/5A50EA77/5A59046B" Ref="#FLG301"  Part="1"
+AR Path="/5A579457/5A569D3F/5A59046B" Ref="#FLG401"  Part="1"
+AR Path="/5A5956FB/5A59046B" Ref="#FLG057"  Part="1"
+AR Path="/5A597FFD/5A59046B" Ref="#FLG063"  Part="1"
+F 0 "#FLG301" H 1250 1225 50  0001 C CNN
 F 1 "PWR_FLAG" H 1250 1300 50  0000 C CNN
 F 2 "" H 1250 1150 50  0001 C CNN
@@
 	1200 1150 1650 1150
 Connection ~ 1250 1150
+$Comp
+L D D401
+U 1 1 5A6334E6
+P 4100 6850
+AR Path="/5A579457/5A569D3F/5A6334E6" Ref="D401"  Part="1"
+AR Path="/5A579457/5A50EA77/5A6334E6" Ref="D301"  Part="1"
+F 0 "D301" H 4100 6950 50  0000 C CNN
+F 1 "D" H 4100 6750 50  0000 C CNN
+F 2 "footprints:D_0603_HandSoldering" H 4100 6850 50  0001 C CNN
+F 3 "" H 4100 6850 50  0001 C CNN
+	1    4100 6850
+	1    0    0    -1
+$EndComp
+Wire Wire Line
+	4250 6850 4250 6600
+Connection ~ 4250 6600
+Text GLabel 3950 6850 0    60   Input ~ 0
+RST
 $EndSCHEMATC
