File: Electrical/Dual/Dual.sch (KiCad schematic (older format))
At the start: 23 parts, among them J101 01x10, J102 01x10, J103 01x04, J104 01x10, J105 02x04, J106 01x10, J107 01x10, J108 01x04, J109 01x04, J110 01x04, J111 01x04, J112 01x04, J113 01x10, J114 01x10

Commit message: Fixed DRC errors
Connections:
- net +5V: now also JP101.1, JP102.1, JP103.1
- net GND: now also J113.10 (Pin_10)
- net Vadj: now also JP105.2, JP106.2, JP107.2
- net uart4_rxd: now also J103.3 (Pin_3)
- net uart4_txd: now also J103.2 (Pin_2)
Changed lines of the file:
@@
 ain_3
 $Comp
-L GND #PWR104
+L GND #PWR01
 U 1 1 5A58DFCA
 P 9900 3900
-F 0 "#PWR104" H 9900 3650 50  0001 C CNN
+F 0 "#PWR01" H 9900 3650 50  0001 C CNN
 F 1 "GND" H 9900 3750 50  0000 C CNN
 F 2 "" H 9900 3900 50  0001 C CNN
@@
 Vadj
 $Comp
-L +5V #PWR105
+L +5V #PWR02
 U 1 1 5A58EE8D
 P 10300 1700
-F 0 "#PWR105" H 10300 1550 50  0001 C CNN
+F 0 "#PWR02" H 10300 1550 50  0001 C CNN
 F 1 "+5V" H 10300 1840 50  0000 C CNN
 F 2 "" H 10300 1700 50  0001 C CNN
@@
 	1    0    0    1
 $EndComp
-Text GLabel 4300 1200 0    60   Input ~ 0
+Text GLabel 4300 1100 0    60   Input ~ 0
 3V3S
 $Comp
-L GND #PWR101
+L GND #PWR03
 U 1 1 5A592273
 P 4300 1550
-F 0 "#PWR101" H 4300 1300 50  0001 C CNN
+F 0 "#PWR03" H 4300 1300 50  0001 C CNN
 F 1 "GND" H 4300 1400 50  0000 C CNN
 F 2 "" H 4300 1550 50  0001 C CNN
@@
 $EndComp
 $Comp
-L GND #PWR102
+L GND #PWR04
 U 1 1 5A594B36
 P 5900 1600
-F 0 "#PWR102" H 5900 1350 50  0001 C CNN
+F 0 "#PWR04" H 5900 1350 50  0001 C CNN
 F 1 "GND" H 5900 1450 50  0000 C CNN
 F 2 "" H 5900 1600 50  0001 C CNN
@@
 3V3S
 $Comp
-L GND #PWR103
+L GND #PWR05
 U 1 1 5A59A43C
 P 9600 6200
-F 0 "#PWR103" H 9600 5950 50  0001 C CNN
+F 0 "#PWR05" H 9600 5950 50  0001 C CNN
 F 1 "GND" H 9600 6050 50  0000 C CNN
 F 2 "" H 9600 6200 50  0001 C CNN
@@
 Wire Wire Line
 	6275 5925 1200 5925
+Connection ~ 10900 2000
+Connection ~ 10900 2500
+Connection ~ 10900 3000
+Connection ~ 10300 3000
+Connection ~ 10300 2500
+Connection ~ 10300 2000
+Connection ~ 9600 6000
+Text Label 4300 1300 2    60   ~ 0
+uart4_rxd
+Text Label 4300 1400 2    60   ~ 0
+uart4_txd
+Wire Wire Line
+	4300 1200 4300 1100
 $EndSCHEMATC

Commit message: Associated footprints. Added some footprint libraries to support.
Parts:
- J101, J102, J104, J106, J107, J113, J114: footprint (none) -> Socket_Strips:Socket_Strip_Straight_1x10_Pitch2.54mm
- J103, J108, J109, J110, J111, J112: footprint (none) -> Socket_Strips:Socket_Strip_Straight_1x04_Pitch2.54mm
- J105: footprint (none) -> Socket_Strips:Socket_Strip_Straight_2x04_Pitch2.54mm
- JP101, JP102, JP103, JP104: value JPMC -> JPNC; footprint (none) -> footprints:JPNC
- JP105, JP106, JP107, JP108: footprint (none) -> footprints:JPNO
- RN101: value R_Pack04 -> 1K2; footprint (none) -> footprints:R_Array_1206x04
Changed lines of the file:
@@
 F 0 "J109" H 9100 2300 50  0000 C CNN
 F 1 "01x04" V 9200 2050 50  0000 C CNN
-F 2 "" H 9100 2100 50  0001 C CNN
+F 2 "Socket_Strips:Socket_Strip_Straight_1x04_Pitch2.54mm" H 9100 2100 50  0001 C CNN
 F 3 "" H 9100 2100 50  0001 C CNN
 	1    9100 2100
@@
 P 9700 1600
 F 0 "RN101" V 9400 1600 50  0000 C CNN
-F 1 "R_Pack04" V 9900 1600 50  0000 C CNN
-F 2 "" V 9975 1600 50  0001 C CNN
+F 1 "1K2" V 9900 1600 50  0000 C CNN
+F 2 "footprints:R_Array_1206x04" V 9975 1600 50  0001 C CNN
 F 3 "" H 9700 1600 50  0001 C CNN
 	1    9700 1600
@@
 F 0 "J110" H 9100 2800 50  0000 C CNN
 F 1 "01x04" V 9200 2550 50  0000 C CNN
-F 2 "" H 9100 2600 50  0001 C CNN
+F 2 "Socket_Strips:Socket_Strip_Straight_1x04_Pitch2.54mm" H 9100 2600 50  0001 C CNN
 F 3 "" H 9100 2600 50  0001 C CNN
 	1    9100 2600
@@
 F 0 "J111" H 9100 3300 50  0000 C CNN
 F 1 "01x04" V 9200 3050 50  0000 C CNN
-F 2 "" H 9100 3100 50  0001 C CNN
+F 2 "Socket_Strips:Socket_Strip_Straight_1x04_Pitch2.54mm" H 9100 3100 50  0001 C CNN
 F 3 "" H 9100 3100 50  0001 C CNN
 	1    9100 3100
@@
 F 0 "J112" H 9100 3800 50  0000 C CNN
 F 1 "01x04" V 9200 3550 50  0000 C CNN
-F 2 "" H 9100 3600 50  0001 C CNN
+F 2 "Socket_Strips:Socket_Strip_Straight_1x04_Pitch2.54mm" H 9100 3600 50  0001 C CNN
 F 3 "" H 9100 3600 50  0001 C CNN
 	1    9100 3600
@@
 P 10400 2000
 F 0 "JP101" H 10425 2075 50  0000 C CNN
-F 1 "JPMC" H 10410 1940 50  0001 C CNN
-F 2 "" H 10400 2000 50  0001 C CNN
+F 1 "JPNC" H 10410 1940 50  0001 C CNN
+F 2 "footprints:JPNC" H 10400 2000 50  0001 C CNN
 F 3 "" H 10400 2000 50  0001 C CNN
 	1    10400 2000
@@
 F 0 "JP105" H 10775 2075 50  0000 C CNN
 F 1 "JPNO" H 10810 1940 50  0001 C CNN
-F 2 "" H 10800 2000 50  0001 C CNN
+F 2 "footprints:JPNO" H 10800 2000 50  0001 C CNN
 F 3 "" H 10800 2000 50  0001 C CNN
 	1    10800 2000
@@
 P 10400 2500
 F 0 "JP102" H 10425 2575 50  0000 C CNN
-F 1 "JPMC" H 10410 2440 50  0001 C CNN
-F 2 "" H 10400 2500 50  0001 C CNN
+F 1 "JPNC" H 10410 2440 50  0001 C CNN
+F 2 "footprints:JPNC" H 10400 2500 50  0001 C CNN
 F 3 "" H 10400 2500 50  0001 C CNN
 	1    10400 2500
@@
 F 0 "JP106" H 10775 2575 50  0000 C CNN
 F 1 "JPNO" H 10810 2440 50  0001 C CNN
-F 2 "" H 10800 2500 50  0001 C CNN
+F 2 "footprints:JPNO" H 10800 2500 50  0001 C CNN
 F 3 "" H 10800 2500 50  0001 C CNN
 	1    10800 2500
@@
 P 10400 3000
 F 0 "JP103" H 10425 3075 50  0000 C CNN
-F 1 "JPMC" H 10410 2940 50  0001 C CNN
-F 2 "" H 10400 3000 50  0001 C CNN
+F 1 "JPNC" H 10410 2940 50  0001 C CNN
+F 2 "footprints:JPNC" H 10400 3000 50  0001 C CNN
 F 3 "" H 10400 3000 50  0001 C CNN
 	1    10400 3000
@@
 F 0 "JP107" H 10775 3075 50  0000 C CNN
 F 1 "JPNO" H 10810 2940 50  0001 C CNN
-F 2 "" H 10800 3000 50  0001 C CNN
+F 2 "footprints:JPNO" H 10800 3000 50  0001 C CNN
 F 3 "" H 10800 3000 50  0001 C CNN
 	1    10800 3000
@@
 P 10400 3500
 F 0 "JP104" H 10425 3575 50  0000 C CNN
-F 1 "JPMC" H 10410 3440 50  0001 C CNN
-F 2 "" H 10400 3500 50  0001 C CNN
+F 1 "JPNC" H 10410 3440 50  0001 C CNN
+F 2 "footprints:JPNC" H 10400 3500 50  0001 C CNN
 F 3 "" H 10400 3500 50  0001 C CNN
 	1    10400 3500
@@
 F 0 "JP108" H 10775 3575 50  0000 C CNN
 F 1 "JPNO" H 10810 3440 50  0001 C CNN
-F 2 "" H 10800 3500 50  0001 C CNN
+F 2 "footprints:JPNO" H 10800 3500 50  0001 C CNN
 F 3 "" H 10800 3500 50  0001 C CNN
 	1    10800 3500
@@
 F 0 "J108" H 7500 1500 50  0000 C CNN
 F 1 "01x04" V 7600 1250 50  0000 C CNN
-F 2 "" H 7500 1300 50  0001 C CNN
+F 2 "Socket_Strips:Socket_Strip_Straight_1x04_Pitch2.54mm" H 7500 1300 50  0001 C CNN
 F 3 "" H 7500 1300 50  0001 C CNN
 	1    7500 1300
@@
 F 0 "J103" H 4500 1600 50  0000 C CNN
 F 1 "01x04" V 4600 1350 50  0000 C CNN
-F 2 "" H 4500 1400 50  0001 C CNN
+F 2 "Socket_Strips:Socket_Strip_Straight_1x04_Pitch2.54mm" H 4500 1400 50  0001 C CNN
 F 3 "" H 4500 1400 50  0001 C CNN
 	1    4500 1400
@@
 F 0 "J102" H 3800 6000 50  0000 C CNN
 F 1 "01x10" H 3800 4900 50  0000 C CNN
-F 2 "" H 3800 5500 50  0001 C CNN
+F 2 "Socket_Strips:Socket_Strip_Straight_1x10_Pitch2.54mm" H 3800 5500 50  0001 C CNN
 F 3 "" H 3800 5500 50  0001 C CNN
 	1    3800 5500
@@
 F 0 "J105" H 5650 1500 50  0000 C CNN
 F 1 "02x04" H 5650 1000 50  0000 C CNN
-F 2 "" H 5600 1300 50  0001 C CNN
+F 2 "Socket_Strips:Socket_Strip_Straight_2x04_Pitch2.54mm" H 5600 1300 50  0001 C CNN
 F 3 "" H 5600 1300 50  0001 C CNN
 	1    5600 1300
@@
 F 0 "J107" H 7400 6000 50  0000 C CNN
 F 1 "01x10" H 7400 4900 50  0000 C CNN
-F 2 "" H 7400 5500 50  0001 C CNN
+F 2 "Socket_Strips:Socket_Strip_Straight_1x10_Pitch2.54mm" H 7400 5500 50  0001 C CNN
 F 3 "" H 7400 5500 50  0001 C CNN
 	1    7400 5500
@@
 F 0 "J101" H 2600 6000 50  0000 C CNN
 F 1 "01x10" H 2600 4900 50  0000 C CNN
-F 2 "" H 2600 5500 50  0001 C CNN
+F 2 "Socket_Strips:Socket_Strip_Straight_1x10_Pitch2.54mm" H 2600 5500 50  0001 C CNN
 F 3 "" H 2600 5500 50  0001 C CNN
 	1    2600 5500
@@
 F 0 "J104" H 5000 6000 50  0000 C CNN
 F 1 "01x10" H 5000 4900 50  0000 C CNN
-F 2 "" H 5000 5500 50  0001 C CNN
+F 2 "Socket_Strips:Socket_Strip_Straight_1x10_Pitch2.54mm" H 5000 5500 50  0001 C CNN
 F 3 "" H 5000 5500 50  0001 C CNN
 	1    5000 5500
@@
 F 0 "J106" H 6200 6000 50  0000 C CNN
 F 1 "01x10" H 6200 4900 50  0000 C CNN
-F 2 "" H 6200 5500 50  0001 C CNN
+F 2 "Socket_Strips:Socket_Strip_Straight_1x10_Pitch2.54mm" H 6200 5500 50  0001 C CNN
 F 3 "" H 6200 5500 50  0001 C CNN
 	1    6200 5500
@@
 F 0 "J113" H 9400 6000 50  0000 C CNN
 F 1 "01x10" H 9400 4900 50  0000 C CNN
-F 2 "" H 9400 5500 50  0001 C CNN
+F 2 "Socket_Strips:Socket_Strip_Straight_1x10_Pitch2.54mm" H 9400 5500 50  0001 C CNN
 F 3 "" H 9400 5500 50  0001 C CNN
 	1    9400 5500
@@
 F 0 "J114" H 10600 6000 50  0000 C CNN
 F 1 "01x10" H 10600 4900 50  0000 C CNN
-F 2 "" H 10600 5500 50  0001 C CNN
+F 2 "Socket_Strips:Socket_Strip_Straight_1x10_Pitch2.54mm" H 10600 5500 50  0001 C CNN
 F 3 "" H 10600 5500 50  0001 C CNN
 	1    10600 5500

Commit message: Fixed issues with socket strips vs pin headers
Parts:
- J101, J102, J104, J106, J107, J113, J114: footprint Socket_Strips:Socket_Strip_Straight_1x10_Pitch2.54mm -> Pin_Headers:Pin_Header_Straight_1x10_Pitch2.54mm
- J103, J108, J109, J110, J111, J112: footprint Socket_Strips:Socket_Strip_Straight_1x04_Pitch2.54mm -> Pin_Headers:Pin_Header_Straight_1x04_Pitch2.54mm
- J105: footprint Socket_Strips:Socket_Strip_Straight_2x04_Pitch2.54mm -> Pin_Headers:Pin_Header_Straight_1x08_Pitch2.54mm
Changed lines of the file:
@@
 F 0 "J109" H 9100 2300 50  0000 C CNN
 F 1 "01x04" V 9200 2050 50  0000 C CNN
-F 2 "Socket_Strips:Socket_Strip_Straight_1x04_Pitch2.54mm" H 9100 2100 50  0001 C CNN
+F 2 "Pin_Headers:Pin_Header_Straight_1x04_Pitch2.54mm" H 9100 2100 50  0001 C CNN
 F 3 "" H 9100 2100 50  0001 C CNN
 	1    9100 2100
@@
 F 0 "J110" H 9100 2800 50  0000 C CNN
 F 1 "01x04" V 9200 2550 50  0000 C CNN
-F 2 "Socket_Strips:Socket_Strip_Straight_1x04_Pitch2.54mm" H 9100 2600 50  0001 C CNN
+F 2 "Pin_Headers:Pin_Header_Straight_1x04_Pitch2.54mm" H 9100 2600 50  0001 C CNN
 F 3 "" H 9100 2600 50  0001 C CNN
 	1    9100 2600
@@
 F 0 "J111" H 9100 3300 50  0000 C CNN
 F 1 "01x04" V 9200 3050 50  0000 C CNN
-F 2 "Socket_Strips:Socket_Strip_Straight_1x04_Pitch2.54mm" H 9100 3100 50  0001 C CNN
+F 2 "Pin_Headers:Pin_Header_Straight_1x04_Pitch2.54mm" H 9100 3100 50  0001 C CNN
 F 3 "" H 9100 3100 50  0001 C CNN
 	1    9100 3100
@@
 F 0 "J112" H 9100 3800 50  0000 C CNN
 F 1 "01x04" V 9200 3550 50  0000 C CNN
-F 2 "Socket_Strips:Socket_Strip_Straight_1x04_Pitch2.54mm" H 9100 3600 50  0001 C CNN
+F 2 "Pin_Headers:Pin_Header_Straight_1x04_Pitch2.54mm" H 9100 3600 50  0001 C CNN
 F 3 "" H 9100 3600 50  0001 C CNN
 	1    9100 3600
@@
 F 0 "J108" H 7500 1500 50  0000 C CNN
 F 1 "01x04" V 7600 1250 50  0000 C CNN
-F 2 "Socket_Strips:Socket_Strip_Straight_1x04_Pitch2.54mm" H 7500 1300 50  0001 C CNN
+F 2 "Pin_Headers:Pin_Header_Straight_1x04_Pitch2.54mm" H 7500 1300 50  0001 C CNN
 F 3 "" H 7500 1300 50  0001 C CNN
 	1    7500 1300
@@
 F 0 "J103" H 4500 1600 50  0000 C CNN
 F 1 "01x04" V 4600 1350 50  0000 C CNN
-F 2 "Socket_Strips:Socket_Strip_Straight_1x04_Pitch2.54mm" H 4500 1400 50  0001 C CNN
+F 2 "Pin_Headers:Pin_Header_Straight_1x04_Pitch2.54mm" H 4500 1400 50  0001 C CNN
 F 3 "" H 4500 1400 50  0001 C CNN
 	1    4500 1400
@@
 F 0 "J102" H 3800 6000 50  0000 C CNN
 F 1 "01x10" H 3800 4900 50  0000 C CNN
-F 2 "Socket_Strips:Socket_Strip_Straight_1x10_Pitch2.54mm" H 3800 5500 50  0001 C CNN
+F 2 "Pin_Headers:Pin_Header_Straight_1x10_Pitch2.54mm" H 3800 5500 50  0001 C CNN
 F 3 "" H 3800 5500 50  0001 C CNN
 	1    3800 5500
@@
 F 0 "J105" H 5650 1500 50  0000 C CNN
 F 1 "02x04" H 5650 1000 50  0000 C CNN
-F 2 "Socket_Strips:Socket_Strip_Straight_2x04_Pitch2.54mm" H 5600 1300 50  0001 C CNN
+F 2 "Pin_Headers:Pin_Header_Straight_1x08_Pitch2.54mm" H 5600 1300 50  0001 C CNN
 F 3 "" H 5600 1300 50  0001 C CNN
 	1    5600 1300
@@
 F 0 "J107" H 7400 6000 50  0000 C CNN
 F 1 "01x10" H 7400 4900 50  0000 C CNN
-F 2 "Socket_Strips:Socket_Strip_Straight_1x10_Pitch2.54mm" H 7400 5500 50  0001 C CNN
+F 2 "Pin_Headers:Pin_Header_Straight_1x10_Pitch2.54mm" H 7400 5500 50  0001 C CNN
 F 3 "" H 7400 5500 50  0001 C CNN
 	1    7400 5500
@@
 F 0 "J101" H 2600 6000 50  0000 C CNN
 F 1 "01x10" H 2600 4900 50  0000 C CNN
-F 2 "Socket_Strips:Socket_Strip_Straight_1x10_Pitch2.54mm" H 2600 5500 50  0001 C CNN
+F 2 "Pin_Headers:Pin_Header_Straight_1x10_Pitch2.54mm" H 2600 5500 50  0001 C CNN
 F 3 "" H 2600 5500 50  0001 C CNN
 	1    2600 5500
@@
 F 0 "J104" H 5000 6000 50  0000 C CNN
 F 1 "01x10" H 5000 4900 50  0000 C CNN
-F 2 "Socket_Strips:Socket_Strip_Straight_1x10_Pitch2.54mm" H 5000 5500 50  0001 C CNN
+F 2 "Pin_Headers:Pin_Header_Straight_1x10_Pitch2.54mm" H 5000 5500 50  0001 C CNN
 F 3 "" H 5000 5500 50  0001 C CNN
 	1    5000 5500
@@
 F 0 "J106" H 6200 6000 50  0000 C CNN
 F 1 "01x10" H 6200 4900 50  0000 C CNN
-F 2 "Socket_Strips:Socket_Strip_Straight_1x10_Pitch2.54mm" H 6200 5500 50  0001 C CNN
+F 2 "Pin_Headers:Pin_Header_Straight_1x10_Pitch2.54mm" H 6200 5500 50  0001 C CNN
 F 3 "" H 6200 5500 50  0001 C CNN
 	1    6200 5500
@@
 F 0 "J113" H 9400 6000 50  0000 C CNN
 F 1 "01x10" H 9400 4900 50  0000 C CNN
-F 2 "Socket_Strips:Socket_Strip_Straight_1x10_Pitch2.54mm" H 9400 5500 50  0001 C CNN
+F 2 "Pin_Headers:Pin_Header_Straight_1x10_Pitch2.54mm" H 9400 5500 50  0001 C CNN
 F 3 "" H 9400 5500 50  0001 C CNN
 	1    9400 5500
@@
 F 0 "J114" H 10600 6000 50  0000 C CNN
 F 1 "01x10" H 10600 4900 50  0000 C CNN
-F 2 "Socket_Strips:Socket_Strip_Straight_1x10_Pitch2.54mm" H 10600 5500 50  0001 C CNN
+F 2 "Pin_Headers:Pin_Header_Straight_1x10_Pitch2.54mm" H 10600 5500 50  0001 C CNN
 F 3 "" H 10600 5500 50  0001 C CNN
 	1    10600 5500

Commit message: Working on layout and routing.
Parts:
- removed J101, J102, J104, J106, J107, J113, J114: 01x10, Pin_Headers:Pin_Header_Straight_1x10_Pitch2.54mm, symbol Conn_01x10_Female
- added J104, J105, J106, J107, J108, J109, J114, J115, J116, J117: 01x03, footprints:Pin_Header_Straight_1x03_Pitch2.54mm_Blank, symbol Conn_01x03_Female
- J102: renamed from J105; footprint Pin_Headers:Pin_Header_Straight_1x08_Pitch2.54mm -> Pin_Headers:Pin_Header_Straight_2x04_Pitch2.54mm
- JP101, JP102, JP103, JP104: footprint footprints:JPNC -> footprints:JPNC_Large
- JP105, JP106, JP107, JP108: footprint footprints:JPNO -> footprints:JPNO_Large
- renumbered J103 to J101, J108 to J103, J109 to J110, J110 to J111, J111 to J112, J112 to J113
Connections:
- net 3V3S: now also J104.2 (Pin_2), J105.2 (Pin_2), J106.2 (Pin_2), J107.2 (Pin_2), J108.2 (Pin_2), J109.2 (Pin_2), J114.2 (Pin_2), J115.2 (Pin_2), J116.2 (Pin_2), J117.2 (Pin_2)
- net GND: now also J104.1 (Pin_1), J105.1 (Pin_1), J106.1 (Pin_1), J107.1 (Pin_1), J108.1 (Pin_1), J109.1 (Pin_1), J114.1 (Pin_1), J115.1 (Pin_1), J116.1 (Pin_1), J117.1 (Pin_1)
- net gpio1_12: now also J104.3 (Pin_3)
- net gpio1_13: now also J105.3 (Pin_3)
- net gpio1_14: now also J106.3 (Pin_3)
- net gpio2_22: now also J107.3 (Pin_3)
- net gpio2_23: now also J108.3 (Pin_3)
- net gpio2_25: now also J109.3 (Pin_3)
- net gpio3_16: now also J114.3 (Pin_3)
- net gpio3_17: now also J115.3 (Pin_3)
- net gpio3_19: now also J116.3 (Pin_3)
- net gpio3_20: now also J117.3 (Pin_3)

Commit message: Completed Dual Stepper Layout. TODO: Via stitching.
Parts:
- added x100: 02x05, Pin_Headers:Pin_Header_Straight_2x05_Pitch2.54mm, symbol Conn_02x05_Odd_Even
- added x101, x113, x125, x137: RoutaCell, footprints:RoutaCellTop, symbol RoutaCell
- added x102, x103, x104, x105, x106, x107, x108, x109, x110, x111: RoutaCell, footprints:RoutaCellLeft, symbol RoutaCell
- added x112: RoutaCell, footprints:RoutaCellBottomLeft, symbol RoutaCell
- added x114, x115, x116, x117, x118, x119, x120, x121, x122, x123, x126, x127, x128, x129, x130, x131, x132, x133, x134, x135, x138, x139, x140, x141, x142, x143, x144, x145, x146, x147: RoutaCell, footprints:RoutaCell, symbol RoutaCell
- added x124, x136, x148: RoutaCell, footprints:RoutaCellBottom, symbol RoutaCell
- added x149: RoutaCell, footprints:RoutaCellTopRight, symbol RoutaCell
- added x150, x151, x152, x153, x154, x155, x156, x157, x158, x159: RoutaCell, footprints:RoutaCellRight, symbol RoutaCell
- added x160: RoutaCell, footprints:RoutaCellBottomRight, symbol RoutaCell
Connections:
- net gpio1_12 is gone; now on net gpio1_13: J104.3 (Pin_3)
- net ehrpwm0A: now also RN101.4 (R4.1); no longer RN101.1 (R1.1)
- net ehrpwm0B: now also RN101.3 (R3.1); no longer RN101.2 (R2.1)
- net ehrpwm1A: now also RN101.2 (R2.1); no longer RN101.3 (R3.1)
- net ehrpwm2B: now also RN101.1 (R1.1); no longer RN101.4 (R4.1)
- net gpio1_13: no longer J105.3 (Pin_3)
- net gpio1_14: now also J105.3 (Pin_3); no longer J106.3 (Pin_3)
- net at J110.1 (Pin_1): now also RN101.5 (R4.2); no longer RN101.8 (R1.2)
- net at J113.1 (Pin_1): now also RN101.8 (R1.2); no longer RN101.5 (R4.2)
- net at RN101.6 (R3.2): now also J111.1 (Pin_1); no longer J112.1 (Pin_1)
- net at RN101.7 (R2.2): now also J112.1 (Pin_1); no longer J111.1 (Pin_1)
- new net: x100.1 (Pin_1), x101.U (Up), x102.U (Up), x103.U (Up), x104.U (Up), x105.U (Up), x106.U (Up), x107.U (Up), x108.U (Up), x109.U (Up), x110.U (Up), x111.U (Up), x112.U (Up)
- new net: x100.10 (Pin_10), x149.D (Down), x150.D (Down), x151.D (Down), x152.D (Down), x153.D (Down), x154.D (Down), x155.D (Down), x156.D (Down), x157.D (Down), x158.D (Down), x159.D (Down), x160.D (Down)
- new net: x100.2 (Pin_2), x101.D (Down), x102.D (Down), x103.D (Down), x104.D (Down), x105.D (Down), x106.D (Down), x107.D (Down), x108.D (Down), x109.D (Down), x110.D (Down), x111.D (Down), x112.D (Down)
- new net: x100.3 (Pin_3), x113.U (Up), x114.U (Up), x115.U (Up), x116.U (Up), x117.U (Up), x118.U (Up), x119.U (Up), x120.U (Up), x121.U (Up), x122.U (Up), x123.U (Up), x124.U (Up)
- new net: x100.4 (Pin_4), x113.D (Down), x114.D (Down), x115.D (Down), x116.D (Down), x117.D (Down), x118.D (Down), x119.D (Down), x120.D (Down), x121.D (Down), x122.D (Down), x123.D (Down), x124.D (Down)
- new net: x100.5 (Pin_5), x125.U (Up), x126.U (Up), x127.U (Up), x128.U (Up), x129.U (Up), x130.U (Up), x131.U (Up), x132.U (Up), x133.U (Up), x134.U (Up), x135.U (Up), x136.U (Up)
- new net: x100.6 (Pin_6), x125.D (Down), x126.D (Down), x127.D (Down), x128.D (Down), x129.D (Down), x130.D (Down), x131.D (Down), x132.D (Down), x133.D (Down), x134.D (Down), x135.D (Down), x136.D (Down)
- new net: x100.7 (Pin_7), x137.U (Up), x138.U (Up), x139.U (Up), x140.U (Up), x141.U (Up), x142.U (Up), x143.U (Up), x144.U (Up), x145.U (Up), x146.U (Up), x147.U (Up), x148.U (Up)
- new net: x100.8 (Pin_8), x137.D (Down), x138.D (Down), x139.D (Down), x140.D (Down), x141.D (Down), x142.D (Down), x143.D (Down), x144.D (Down), x145.D (Down), x146.D (Down), x147.D (Down), x148.D (Down)
- new net: x100.9 (Pin_9), x149.U (Up), x150.U (Up), x151.U (Up), x152.U (Up), x153.U (Up), x154.U (Up), x155.U (Up), x156.U (Up), x157.U (Up), x158.U (Up), x159.U (Up), x160.U (Up)
- new net gpio1_20: J106.3 (Pin_3)
Other:
- note added: "Prototyping Area"
